File: Frohne/pcm1808.kicad_sch (KiCad schematic)
At the start: 26 parts, among them J1 ADC IN, U2 PCM1808PWR, X2 YC24.576MUBCE2O

Commit message: Fixed a few schematic errors.
Parts:
- TP1, TP2: footprint TestPoint:TestPoint_THTPad_D1.0mm_Drill0.5mm -> TestPoint:TestPoint_THTPad_D1.5mm_Drill0.7mm
Changed lines of the file:
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@@
 			)
 		)
-		(property "Footprint" "TestPoint:TestPoint_THTPad_D1.0mm_Drill0.5mm"
+		(property "Footprint" "TestPoint:TestPoint_THTPad_D1.5mm_Drill0.7mm"
 			(at 86.36 67.31 0)
 			(effects
@@
 			)
 		)
-		(property "Footprint" "TestPoint:TestPoint_THTPad_D1.0mm_Drill0.5mm"
+		(property "Footprint" "TestPoint:TestPoint_THTPad_D1.5mm_Drill0.7mm"
 			(at 76.2 69.85 0)
 			(effects
