File: Frohne/qsd-sdr.kicad_sch (KiCad schematic)
At the start: 51 parts, among them J11 SDR ANT, J12 SDR Out, U5 OPA1612AxD, U7 SN74CBT3253, U8 OPA1612AxD

Commit message: 328 warnings
Parts:
- Je3: now not fitted
Changed lines of the file:
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@@
 		(in_bom yes)
 		(on_board yes)
-		(dnp no)
+		(dnp yes)
 		(fields_autoplaced yes)
 		(property "Reference" "Je3"
