File: Frohne/Frohne.kicad_sch (KiCad schematic)
At the start: 6 parts

Commit message: Fixed a few more things and started routing.
Other:
- sheet PCM1808 ports: added SKCI; removed LO_CLK
Changed lines of the file:
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@@
 			)
 		)
-		(pin "LO_CLK" input
+		(pin "SKCI" input
 			(at 62.23 176.53 180)
 			(effects
