File: Frohne/VDDA.kicad_sch (KiCad schematic)
At the start: 30 parts, among them J5 Conn_01x02, Q1 AO3401A, U6 L78M05ABDT-TR

Commit message: 328 warnings
Parts:
- J5: now not fitted
Changed lines of the file:
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@@
 		(in_bom yes)
 		(on_board yes)
-		(dnp no)
+		(dnp yes)
 		(fields_autoplaced yes)
 		(property "Reference" "J5"
