File: Module_JaronGarbi/Module_JaronGarbi.kicad_pcb (KiCad board)
At the start: 4 copper layers, 9 parts, among them J1 Conn_01x03

Commit message: No Errors No Warnings
Some were excluded.
Parts:
- removed D10, D8, D9: WS2812B, PCM_JLCPCB:LED_WS2812B_PLCC4_5.0x5.0mm_P3.2mm
- added D2: WS2812B, PCM_JLCPCB:LED_WS2812B_PLCC4_5.0x5.0mm_P3.2mm, F.Cu at (179.3, 88.5)
- added D3: WS2812B, PCM_JLCPCB:LED_WS2812B_PLCC4_5.0x5.0mm_P3.2mm, F.Cu at (186.2, 88.5)
- added D4: WS2812B, PCM_JLCPCB:LED_WS2812B_PLCC4_5.0x5.0mm_P3.2mm, F.Cu at (193.1, 88.5)
- renumbered C62 to C1, C64 to C2, C65 to C3, C67 to C4, D11 to D1
Connections:
- net +4.7V renamed +3.3V
Routing:
- net +3.3V: track 42.8 -> 24.1 mm
- net Net-(D2-DOUT): track 0.00 -> 6.89 mm
- net Net-(D10-DOUT): track 6.89 -> 0.00 mm
- net Net-(D8-DIN): track 6.87 -> 0.00 mm
- net Net-(D3-DOUT): track 0.00 -> 6.87 mm
