File: Module_JaronGarbi/Module_JaronGarbi.kicad_sch (KiCad schematic)
At the start: 9 parts, among them J1 Conn_01x03

Commit message: Imported Student Parts
Not using Project Instances yet.
Parts:
- removed D10, D8, D9: WS2812B, PCM_JLCPCB:LED_WS2812B_PLCC4_5.0x5.0mm_P3.2mm, symbol PCM_JLCPCB-Extended:LED, WS2812B, 5050
- added D? (x3): WS2812B, PCM_JLCPCB:LED_WS2812B_PLCC4_5.0x5.0mm_P3.2mm, symbol PCM_JLCPCB-Extended:LED, WS2812B, 5050
- renumbered C65 to C?, C67 to C?, C64 to C?, C62 to C?, D11 to D?, J1 to J?
Connections:
- net GND: now also D?.3 (VSS), D?.3 (VSS), D?.3 (VSS)
- net at D?.2 (DOUT): now also D?.4 (DIN)
- net at J?.2 (Pin_2): now also D?.2 (DOUT)
- net +4.7V renamed +3.3V
- net +3.3V: now also D?.1 (VDD), D?.1 (VDD), D?.1 (VDD)
- new net: D?.2 (DOUT), D?.4 (DIN) (x2)

Commit message: Going to school.
Parts:
- gave numbers to parts that had none: 9
Changed lines of the file:
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@@
 		(dnp no)
 		(fields_autoplaced yes)
-		(property "Reference" "#PWR?"
+		(property "Reference" "#PWR0138"
 			(at 177.8 115.57 0)
 			(effects
@@
 			(project "Module_Template"
 				(path "/c12dc015-e6cb-468c-8de4-269c3106de0e/3aa3dec0-5ad1-4c27-a945-0a713a163b16"
-					(reference "#PWR?")
+					(reference "#PWR0138")
 					(unit 1)
 				)
@@
 		(dnp no)
 		(fields_autoplaced yes)
-		(property "Reference" "#PWR?"
+		(property "Reference" "#PWR0127"
 			(at 57.15 97.79 0)
 			(effects
@@
 			(project "Module_Template"
 				(path "/c12dc015-e6cb-468c-8de4-269c3106de0e/3aa3dec0-5ad1-4c27-a945-0a713a163b16"
-					(reference "#PWR?")
+					(reference "#PWR0127")
 					(unit 1)
 				)
@@
 		(dnp no)
 		(fields_autoplaced yes)
-		(property "Reference" "#PWR?"
+		(property "Reference" "#PWR0139"
 			(at 195.58 114.3 0)
 			(effects
@@
 			(project "Intro-to-CAD-2026"
 				(path "/c12dc015-e6cb-468c-8de4-269c3106de0e/3aa3dec0-5ad1-4c27-a945-0a713a163b16"
-					(reference "#PWR?")
+					(reference "#PWR0139")
 					(unit 1)
 				)
@@
 		(dnp no)
 		(fields_autoplaced yes)
-		(property "Reference" "#PWR?"
+		(property "Reference" "#PWR0128"
 			(at 71.12 95.25 0)
 			(effects
@@
 			(project "Intro-to-CAD-2026"
 				(path "/c12dc015-e6cb-468c-8de4-269c3106de0e/3aa3dec0-5ad1-4c27-a945-0a713a163b16"
-					(reference "#PWR?")
+					(reference "#PWR0128")
 					(unit 1)
 				)
@@
 		(dnp no)
 		(fields_autoplaced yes)
-		(property "Reference" "#PWR?"
+		(property "Reference" "#PWR0135"
 			(at 142.24 115.57 0)
 			(effects
@@
 			(project "Module_Template"
 				(path "/c12dc015-e6cb-468c-8de4-269c3106de0e/3aa3dec0-5ad1-4c27-a945-0a713a163b16"
-					(reference "#PWR?")
+					(reference "#PWR0135")
 					(unit 1)
 				)
@@
 		(dnp no)
 		(fields_autoplaced yes)
-		(property "Reference" "#PWR?"
+		(property "Reference" "#PWR0137"
 			(at 177.8 95.25 0)
 			(effects
@@
 			(project "Intro-to-CAD-2026"
 				(path "/c12dc015-e6cb-468c-8de4-269c3106de0e/3aa3dec0-5ad1-4c27-a945-0a713a163b16"
-					(reference "#PWR?")
+					(reference "#PWR0137")
 					(unit 1)
 				)
@@
 		(dnp no)
 		(fields_autoplaced yes)
-		(property "Reference" "#PWR?"
+		(property "Reference" "#PWR0130"
 			(at 92.71 97.79 0)
 			(effects
@@
 			(project "Module_Template"
 				(path "/c12dc015-e6cb-468c-8de4-269c3106de0e/3aa3dec0-5ad1-4c27-a945-0a713a163b16"
-					(reference "#PWR?")
+					(reference "#PWR0130")
 					(unit 1)
 				)
@@
 		(dnp no)
 		(fields_autoplaced yes)
-		(property "Reference" "#PWR?"
+		(property "Reference" "#PWR0133"
 			(at 128.27 97.79 0)
 			(effects
@@
 			(project "Module_Template"
 				(path "/c12dc015-e6cb-468c-8de4-269c3106de0e/3aa3dec0-5ad1-4c27-a945-0a713a163b16"
-					(reference "#PWR?")
+					(reference "#PWR0133")
 					(unit 1)
 				)
@@
 		(dnp no)
 		(fields_autoplaced yes)
-		(property "Reference" "C?"
+		(property "Reference" "C70"
 			(at 134.62 82.55 90)
 			(effects
@@
 			(project "Module_Template"
 				(path "/c12dc015-e6cb-468c-8de4-269c3106de0e/3aa3dec0-5ad1-4c27-a945-0a713a163b16"
-					(reference "C?")
+					(reference "C70")
 					(unit 1)
 				)
@@
 		(dnp no)
 		(fields_autoplaced yes)
-		(property "Reference" "#PWR?"
+		(property "Reference" "#PWR0140"
 			(at 210.82 107.95 0)
 			(effects
@@
 			(project "Module_Template"
 				(path "/c12dc015-e6cb-468c-8de4-269c3106de0e/3aa3dec0-5ad1-4c27-a945-0a713a163b16"
-					(reference "#PWR?")
+					(reference "#PWR0140")
 					(unit 1)
 				)
@@
 		(dnp no)
 		(fields_autoplaced yes)
-		(property "Reference" "#PWR?"
+		(property "Reference" "#PWR0129"
 			(at 71.12 115.57 0)
 			(effects
@@
 			(project "Module_Template"
 				(path "/c12dc015-e6cb-468c-8de4-269c3106de0e/3aa3dec0-5ad1-4c27-a945-0a713a163b16"
-					(reference "#PWR?")
+					(reference "#PWR0129")
 					(unit 1)
 				)
@@
 		(dnp no)
 		(fields_autoplaced yes)
-		(property "Reference" "#PWR?"
+		(property "Reference" "#PWR0136"
 			(at 163.83 97.79 0)
 			(effects
@@
 			(project "Module_Template"
 				(path "/c12dc015-e6cb-468c-8de4-269c3106de0e/3aa3dec0-5ad1-4c27-a945-0a713a163b16"
-					(reference "#PWR?")
+					(reference "#PWR0136")
 					(unit 1)
 				)
@@
 		(dnp no)
 		(fields_autoplaced yes)
-		(property "Reference" "#PWR?"
+		(property "Reference" "#PWR0132"
 			(at 106.68 115.57 0)
 			(effects
@@
 			(project "Module_Template"
 				(path "/c12dc015-e6cb-468c-8de4-269c3106de0e/3aa3dec0-5ad1-4c27-a945-0a713a163b16"
-					(reference "#PWR?")
+					(reference "#PWR0132")
 					(unit 1)
 				)
@@
 		(dnp no)
 		(fields_autoplaced yes)
-		(property "Reference" "D?"
+		(property "Reference" "D11"
 			(at 189.23 95.1798 0)
 			(effects
@@
 			(project "Intro-to-CAD-2026"
 				(path "/c12dc015-e6cb-468c-8de4-269c3106de0e/3aa3dec0-5ad1-4c27-a945-0a713a163b16"
-					(reference "D?")
+					(reference "D11")
 					(unit 1)
 				)
@@
 		(dnp no)
 		(fields_autoplaced yes)
-		(property "Reference" "C?"
+		(property "Reference" "C71"
 			(at 170.18 82.55 90)
 			(effects
@@
 			(project "Module_Template"
 				(path "/c12dc015-e6cb-468c-8de4-269c3106de0e/3aa3dec0-5ad1-4c27-a945-0a713a163b16"
-					(reference "C?")
+					(reference "C71")
 					(unit 1)
 				)
@@
 		(dnp no)
 		(fields_autoplaced yes)
-		(property "Reference" "C?"
+		(property "Reference" "C69"
 			(at 99.06 82.55 90)
 			(effects
@@
 			(project "Module_Template"
 				(path "/c12dc015-e6cb-468c-8de4-269c3106de0e/3aa3dec0-5ad1-4c27-a945-0a713a163b16"
-					(reference "C?")
+					(reference "C69")
 					(unit 1)
 				)
@@
 		(dnp no)
 		(fields_autoplaced yes)
-		(property "Reference" "#PWR?"
+		(property "Reference" "#PWR0131"
 			(at 106.68 95.25 0)
 			(effects
@@
 			(project "Intro-to-CAD-2026"
 				(path "/c12dc015-e6cb-468c-8de4-269c3106de0e/3aa3dec0-5ad1-4c27-a945-0a713a163b16"
-					(reference "#PWR?")
+					(reference "#PWR0131")
 					(unit 1)
 				)
@@
 		(dnp no)
 		(fields_autoplaced yes)
-		(property "Reference" "D?"
+		(property "Reference" "D10"
 			(at 153.67 95.1798 0)
 			(effects
@@
 			(project "Intro-to-CAD-2026"
 				(path "/c12dc015-e6cb-468c-8de4-269c3106de0e/3aa3dec0-5ad1-4c27-a945-0a713a163b16"
-					(reference "D?")
+					(reference "D10")
 					(unit 1)
 				)
@@
 		(dnp no)
 		(fields_autoplaced yes)
-		(property "Reference" "D?"
+		(property "Reference" "D9"
 			(at 118.11 95.1798 0)
 			(effects
@@
 			(project "Intro-to-CAD-2026"
 				(path "/c12dc015-e6cb-468c-8de4-269c3106de0e/3aa3dec0-5ad1-4c27-a945-0a713a163b16"
-					(reference "D?")
+					(reference "D9")
 					(unit 1)
 				)
@@
 		(dnp no)
 		(fields_autoplaced yes)
-		(property "Reference" "J?"
+		(property "Reference" "J14"
 			(at 223.52 106.6799 0)
 			(effects
@@
 			(project ""
 				(path "/c12dc015-e6cb-468c-8de4-269c3106de0e/3aa3dec0-5ad1-4c27-a945-0a713a163b16"
-					(reference "J?")
+					(reference "J14")
 					(unit 1)
 				)
@@
 		(dnp no)
 		(fields_autoplaced yes)
-		(property "Reference" "#PWR?"
+		(property "Reference" "#PWR0134"
 			(at 142.24 95.25 0)
 			(effects
@@
 			(project "Intro-to-CAD-2026"
 				(path "/c12dc015-e6cb-468c-8de4-269c3106de0e/3aa3dec0-5ad1-4c27-a945-0a713a163b16"
-					(reference "#PWR?")
+					(reference "#PWR0134")
 					(unit 1)
 				)
@@
 		(dnp no)
 		(fields_autoplaced yes)
-		(property "Reference" "D?"
+		(property "Reference" "D8"
 			(at 82.55 95.1798 0)
 			(effects
@@
 			(project "Module_Template"
 				(path "/c12dc015-e6cb-468c-8de4-269c3106de0e/3aa3dec0-5ad1-4c27-a945-0a713a163b16"
-					(reference "D?")
+					(reference "D8")
 					(unit 1)
 				)
@@
 		(dnp no)
 		(fields_autoplaced yes)
-		(property "Reference" "C?"
+		(property "Reference" "C68"
 			(at 63.5 82.55 90)
 			(effects
@@
 			(project "Module_Template"
 				(path "/c12dc015-e6cb-468c-8de4-269c3106de0e/3aa3dec0-5ad1-4c27-a945-0a713a163b16"
-					(reference "C?")
-					(unit 1)
-				)
+					(reference "C68")
+					(unit 1)
+				)

Commit message: Replaced Jaron's LEDs
They were only for Standard Boards.
Parts:
- D10, D11, D8, D9: value WS2812B -> XL-0807RGBC-2812B; footprint PCM_JLCPCB:LED_WS2812B_PLCC4_5.0x5.0mm_P3.2mm -> Intro_to_CAD:C3646929e; LCSC C22461793 -> C3646929

Commit message: Fixed pinout error on LEDs.
Connections:
- net +3.3V: now also D10.4 (VDD), D11.4 (VDD), D8.4 (VDD), D9.4 (VDD); no longer D10.1 (VDD), D11.1 (VDD), D8.1 (VDD), D9.1 (VDD)
- net GND: now also D10.2 (GND), D11.2 (GND), D8.2 (GND), D9.2 (GND); no longer D10.3 (VSS), D11.3 (VSS), D8.3 (VSS), D9.3 (VSS)
- net RGB_DIN: now also D8.3 (DIN); no longer D8.4 (DIN)
- net at J14.2 (Pin_2): now also D11.1 (DOUT); no longer D11.2 (DOUT)
- new net: D10.3 (DIN), D9.1 (DOUT)
- new net: D8.1 (DOUT), D9.3 (DIN)
- new net: D10.1 (DOUT), D11.3 (DIN)

Commit message: Placed the second ADC
Parts:
- C68, C69, C70, C71: Manufacturer YAGEO -> (none)
Changed lines of the file:
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@@
-			)
-		)
-		(property "Manufacturer" "YAGEO"
-			(at 134.62 91.44 0)
-			(hide yes)
-			(show_name no)
-			(do_not_autoplace no)
-			(effects
-				(font
-					(size 1.27 1.27)
-				)
 			)
 		)
@@
 			)
 		)
-		(property "Manufacturer" "YAGEO"
-			(at 170.18 91.44 0)
-			(hide yes)
-			(show_name no)
-			(do_not_autoplace no)
-			(effects
-				(font
-					(size 1.27 1.27)
-				)
-			)
-		)
 		(property "Part" "CC0603KRX7R9BB104"
 			(at 170.18 91.44 0)
@@
 			)
 		)
-		(property "Manufacturer" "YAGEO"
-			(at 99.06 91.44 0)
-			(hide yes)
-			(show_name no)
-			(do_not_autoplace no)
-			(effects
-				(font
-					(size 1.27 1.27)
-				)
-			)
-		)
 		(property "Part" "CC0603KRX7R9BB104"
 			(at 99.06 91.44 0)
@@
 			(at 63.5 91.44 0)
 			(hide yes)
-			(show_name no)
-			(do_not_autoplace no)
-			(effects
-				(font
-					(size 1.27 1.27)
-				)
-			)
-		)
-		(property "Manufacturer" "YAGEO"
-			(at 63.5 91.44 0)
-			(hide yes)
