File: VDDA.kicad_sch (KiCad schematic)
At the start: 30 parts, among them J5 Conn_01x02, Q1 AO3401A, U6 L78M05ABDT-TR

Commit message: Initial v0.2
Fixed SCL-SDA swap, 3V3 on encoder, and 3D models for Kicad 10
Parts:
- FB2, FB5, FB6, JP2: value ~ -> (none)

Commit message: Updated errors
Other:
- note added: "+5V Clean Analog Supply option which also provides a way to power the Pico if it has no USB connection. Beware! Do not use this until you have fixed Q1's wiring problem or use only 5V for the external DC input. Once the Q1 is fixed you can disconnect the VAH jumper to the push-pull DAC amp and then connect +12V here if you like."
- note added: "We need to reverse the drain and source on Q1."
- note removed: "+12V Clean Analog Supply option which also provides a way to power the Pico if it has no USB connection."
Changed lines of the file:
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@@
+		)
+	)
+	(text "We need to reverse the drain and source on Q1."
+		(exclude_from_sim no)
+		(at 89.916 131.064 0)
+		(effects
+			(font
+				(size 1.27 1.27)
+				(color 255 4 41 1)
+			)
 		)
 	)
@@
 		)
 	)
-	(text "+12V Clean \nAnalog Supply\noption which\nalso provides\na way to power\nthe Pico if it\nhas no USB \nconnection."
+	(text "+5V Clean \nAnalog Supply\noption which\nalso provides\na way to power\nthe Pico if it\nhas no USB \nconnection.\nBeware!  Do not\nuse this until you\nhave fixed Q1's \nwiring problem or \nuse only 5V for the\nexternal DC input.\nOnce the Q1 is fixed\nyou can disconnect\nthe VAH jumper to\nthe push-pull DAC\namp and then connect\n+12V here if you like."
 		(exclude_from_sim no)
-		(at 88.9 46.482 0)
+		(at 76.708 48.514 0)
 		(effects
 			(font
 				(size 1.27 1.27)
+				(color 255 2 79 1)
 			)
+			(justify left)
 		)
 	)
