File: Intro-to-CAD-2026.kicad_pcb (KiCad board)
At the start: 4 copper layers, 100 x 100 mm, 335 parts, among them J1 ADC IN, J10 Conn_01x20_Socket, J11 SDR ANT, J12 SDR Out, J13 Micro_SD-TF_PUSH, J14 Conn_01x03, J15 OLED, J16 3.5mm_Jack, J17 Screw_Terminal_01x02, J18 Screw_Terminal_01x02, J2 Conn_02x20_Counter_Clockwise, J3 Conn_02x20_Counter_Clockwise, J4 Conn_01x20_Socket, J5 Conn_01x02, J6 HC-SR04, J7 Conn_01x01_Pin, J9 3.5mm_Jack, Q1 AO3401A, Q2 FMMT591, Q3 FMMT491, Q4 FMMT491, Q5 FMMT591, SW1 RotaryEncoder_Switch_MP, U1 CJC4334H, U10 TC118S, U11 SN74LVC74ADR, U2 PCM1808PWR, U3 Pico, U4 MS5351M, U5 OPA1612AxD, U6 L78M05ABDT-TR, U7 SN74CBT3253DBQR, U8 OPA1612AxD, U9 OPA1612AxD, X1 YC24.576MUBCE2O

Commit message: Saved.
Parts:
- moved C89 120.5 mm to (140.7, 112.9), turned to 180 degrees
- moved TP27 119.0 mm to (145.3, 109.9)
- moved C82 117.9 mm to (137.8, 129.2)
- moved R25 117.2 mm to (144.7, 102.1)
- moved R73 117.2 mm to (144.7, 105.0)
- moved R10 116.0 mm to (144.9, 93.8), turned to 180 degrees
- moved R24 115.6 mm to (145.0, 95.9), turned to 180 degrees
- moved FB9 114.9 mm to (145.4, 107.2), turned to 180 degrees
- moved C90 114.6 mm to (140.7, 108.5), turned to 180 degrees
- moved C81 110.1 mm to (133.4, 129.7), turned to 180 degrees
- moved C88 107.9 mm to (144.6, 99.7), turned to 0 degrees
- moved C87 102.7 mm to (144.9, 97.5)
- moved C85 102.7 mm to (144.9, 85.7)
- moved C83 101.2 mm to (126.9, 120.7), turned to 90 degrees
- moved C86 100.8 mm to (144.6, 88.1)
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Routing:
- net Net-(e10-EN): track 0.00 -> 61.7 mm
- net VDDA: track 55.9 -> 100.0 mm, vias 3 -> 7
- net Net-(TR1-C_RX): track 16.4 -> 34.5 mm, vias 0 -> 2
- net VAO: track 6.61 -> 23.0 mm, vias 0 -> 2
- net Net-(C87-Pad1): track 0.00 -> 10.1 mm
- net Net-(e10-SENSE/ADJ): track 0.00 -> 6.44 mm
- net Net-(Q1-S): track 3.22 -> 8.13 mm
- net Net-(C42-Pad1): track 5.69 -> 9.03 mm
- net Net-(D1-Pad1): track 2.79 -> 4.41 mm
- net /Si5351a/3.3VAO: track 55.3 -> 54.3 mm

Commit message: edits
Parts:
- added C95: 100uF, PCM_JLCPCB:C_CASE-B-3528-21(mm), F.Cu at (160.4, 112.7)
- added C96: 100uF, PCM_JLCPCB:C_CASE-B-3528-21(mm), F.Cu at (155.1, 117.1)
- added C97: 100nF, PCM_JLCPCB:C_0805, F.Cu at (160.5, 124.7)
- added C98: 100nF, PCM_JLCPCB:C_0805, F.Cu at (163.4, 117.1)
- moved JP3 0.61 mm to (154.9, 120.6), turned to 180 degrees
- moved C63 0.37 mm to (156.2, 122.9)
Connections:
- C43 pad 1: VAH -> Net-(JP2-A)
- D3 pad 2: VAH -> Net-(JP2-A)
- JP2 pad 1: VAH -> Net-(JP2-A)
- U6 pad 3: VAH -> Net-(JP2-A)
- e2 pad 2: VAH -> +4.7V
Routing:
- net /Si5351a/3.3VAO: track 54.3 -> 3.67 mm, vias 8 -> 0
- net VDDA: track 100.0 -> 69.4 mm, vias 7 -> 5
- net /DAC/VA/2: track 14.8 -> 29.1 mm
- net VAH: track 10.9 -> 0.00 mm, vias 1 -> 0
- net Net-(JP2-A): track 0.00 -> 10.9 mm, vias 0 -> 1
- net VAO: track 23.0 -> 25.9 mm

Commit message: Added CJC5340
Parts:
- removed JP5: MCLK, Jumper:SolderJumper-2_P1.3mm_Open_RoundedPad1.0x1.5mm
- removed e9: EX_CLK, Jumper:SolderJumper-2_P1.3mm_Bridged_RoundedPad1.0x1.5mm
- added C104: 10uF, PCM_JLCPCB:C_CASE-A-3216-18(mm), F.Cu at (76.7, 53.0)
- added C106: 100nF, PCM_JLCPCB:C_0805, F.Cu at (71.6, 53.0)
- added C108: 10uF, PCM_JLCPCB:C_CASE-A-3216-18(mm), F.Cu at (76.7, 56.2)
- added C109: 100nF, PCM_JLCPCB:C_0805, F.Cu at (71.6, 56.0)
- added C110: 100nF, PCM_JLCPCB:C_0805, F.Cu at (71.6, 59.1)
- added C112: 100nF, PCM_JLCPCB:C_0805, F.Cu at (71.6, 62.1)
- added C113: 10uF, PCM_JLCPCB:C_CASE-A-3216-18(mm), F.Cu at (76.7, 59.3)
- added C114: 100nF, PCM_JLCPCB:C_0805, F.Cu at (71.6, 65.2)
- added C99: 100uF, PCM_JLCPCB:C_CASE-B-3528-21(mm), F.Cu at (82.6, 53.6)
- added JP11: Clock Select, Jumper:SolderJumper-3_P1.3mm_Bridged12_RoundedPad1.0x1.5mm_NumberLabels, F.Cu at (92.2, 56.8)
- added JP12: Clock Select, Jumper:SolderJumper-3_P1.3mm_Bridged12_RoundedPad1.0x1.5mm_NumberLabels, F.Cu at (92.2, 60.3)
- added JP13: Clock Select, Jumper:SolderJumper-3_P1.3mm_Bridged12_RoundedPad1.0x1.5mm_NumberLabels, F.Cu at (92.2, 63.9)
- added JP14: Clock Select, Jumper:SolderJumper-3_P1.3mm_Bridged12_RoundedPad1.0x1.5mm_NumberLabels, F.Cu at (92.2, 67.4)
- added R75: 10kΩ, PCM_JLCPCB:R_0402, F.Cu at (81.0, 56.7)
- added R76: 33Ω, PCM_JLCPCB:R_0805, F.Cu at (91.6, 72.7)
- added R78: 33Ω, PCM_JLCPCB:R_0805, F.Cu at (85.1, 62.4)
- added R79: 33Ω, PCM_JLCPCB:R_0805, F.Cu at (85.1, 65.3)
- added R81: 5.1Ω, PCM_JLCPCB:R_0805, F.Cu at (85.1, 68.3)
- added U13: ~, Package_SO:TSSOP-16_4.4x5mm_P0.65mm, F.Cu at (78.6, 64.2)
- JP6: value MCLK -> Clock Select; footprint Jumper:SolderJumper-2_P1.3mm_Open_RoundedPad1.0x1.5mm -> Jumper:SolderJumper-3_P1.3mm_Bridged12_RoundedPad1.0x1.5mm_NumberLabels; moved to F.Cu
- moved C26 101.3 mm to (199.4, 95.8), turned to -90 degrees
- moved R71 97.9 mm to (197.7, 95.8), turned to 90 degrees
- moved e8 89.7 mm to (192.3, 98.5), turned to 0 degrees
- moved C49 89.7 mm to (188.8, 105.0), turned to 0 degrees
- moved J16 89.6 mm to (191.3, 100.5), turned to -90 degrees
- moved C53 86.8 mm to (191.7, 96.0), turned to 0 degrees
- moved R32 84.8 mm to (183.3, 108.4), turned to -90 degrees
- moved R22 83.7 mm to (185.2, 105.0), turned to 0 degrees
- moved C46 79.8 mm to (179.8, 108.5), turned to 0 degrees
- moved C45 77.6 mm to (180.9, 105.5), turned to 0 degrees
- moved C24 77.3 mm to (183.8, 101.3), turned to 0 degrees
- moved FB7 76.0 mm to (181.5, 103.6), turned to 0 degrees
- moved C25 74.1 mm to (183.7, 98.3), turned to 0 degrees
- moved R33 73.2 mm to (184.3, 96.2), turned to 0 degrees
- moved C12 72.0 mm to (180.4, 101.7), turned to 0 degrees
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Connections:
- net Net-(U2-VINL) renamed /AUD_L
- net Net-(U2-VINR) renamed /AUD_R
- JP27 pad 1: /Raspberry_Pi_Pico/GPIO26_ADC0 -> /ECHO
- JP28 pad 1: /RGB_DIN -> /TRIG
- JP29 pad 1: /BTN -> /ANG_A
- JP30 pad 1: /ECHO -> /ANG_B
- JP31 pad 1: /TRIG -> /RGB_DIN
- JP32 pad 1: /ANG_A -> /SDIN
- JP33 pad 1: /ANG_B -> /LRCK
- JP34 pad 1: /WS -> /SCLK
- JP6 pad 1: /MCLK -> /EX_CLK
- JP74 pad 2: /SCLK -> /SD2
- JP75 pad 2: /LRCK -> /BCK2
- JP76 pad 2: /MCLK -> /WS2
- JP77 pad 2: /SDIN -> /DATA
- JP78 pad 2: /FMT -> /BCK
- JP79 pad 2: /MD1 -> /WS
- JP82 pad 2: /DATA -> /BTN
- JP83 pad 2: /BCK -> /PICO_MCLK
- R34 pad 2: Net-(JP5-B) -> Net-(X1-OUT)
- R35 pad 1: Net-(JP5-A) -> Net-(X1-OUT)
- R35 pad 2: /CMOS Oscillator/SCKI -> /SCKI2
- R36 pad 2: Net-(JP5-A) -> Net-(X1-OUT)
- U2 pad 11: /MD1 -> /MD1/M1
- U2 pad 12: /FMT -> /FMT/M0
- U2 pad 6: /CMOS Oscillator/SCKI -> /SCKI1
- X1 pad 3: Net-(JP5-A) -> Net-(X1-OUT)
Routing:
- net /SW_C: track 107.8 -> 10.3 mm, vias 2 -> 0
- net /RGB_DIN: track 56.9 -> 0.00 mm, vias 3 -> 0
- net /WS: track 48.2 -> 0.00 mm, vias 1 -> 0
- net /TRIG: track 42.3 -> 0.00 mm, vias 1 -> 0
- net /ECHO: track 41.3 -> 0.00 mm, vias 1 -> 0
- net /EX_CLK: track 30.3 -> 2.77 mm, vias 1 -> 0
- net /FMT: track 20.1 -> 0.00 mm, vias 3 -> 0
- net /BTN: track 21.8 -> 2.71 mm, vias 1 -> 0
- net Net-(C60-Pad2): track 17.0 -> 0.00 mm, vias 2 -> 0
- net /MD1: track 15.9 -> 0.00 mm, vias 1 -> 0
- net /ANG_A: track 34.3 -> 19.1 mm, vias 1 -> 0
- net /BCK: track 12.0 -> 0.00 mm, vias 1 -> 0
- net /ANG_B: track 24.9 -> 13.3 mm, vias 1 -> 0
- net GND: track 168.3 -> 157.4 mm, vias 9 -> 8
- net Net-(C24-Pad2): track 9.81 -> 0.00 mm
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
Commit message: More edits....
Parts:
- JP11: value Clock Select -> M0; moved to B.Cu
- JP12: value Clock Select -> M1; moved to B.Cu
- JP13: value Clock Select -> FMT; moved to B.Cu
- JP14: value Clock Select -> MD1; moved to B.Cu
- JP6: value Clock Select -> DAC MCLK; moved to B.Cu
- moved U13 45.7 mm to (123.9, 58.6), turned to -90 degrees
- moved R76 37.6 mm to (125.9, 88.0), turned to -90 degrees
- moved C84 1.85 mm to (123.0, 89.3)
- moved C9 1.30 mm to (120.3, 86.8)
- turned JP11 to 180 degrees
- turned JP12 to 180 degrees
- turned JP13 to 180 degrees
- turned JP14 to 180 degrees
- turned JP6 to 180 degrees
Routing:
- net /SCL: track 48.0 -> 0.00 mm, vias 1 -> 0
- net /SDA: track 42.9 -> 0.00 mm, vias 1 -> 0
- net /OSC_SCL: track 53.6 -> 19.9 mm, vias 3 -> 2
- net /OSC_SDA: track 60.7 -> 39.5 mm
- net (no net): track 7.53 -> 0.00 mm
- net /EX_CLK: track 2.77 -> 0.00 mm
- net /DAC/MCLK: track 2.66 -> 0.00 mm
- net Net-(X1-OUT): track 5.46 -> 7.34 mm, vias 2 -> 0
- net VDDA: track 69.4 -> 70.6 mm
Other:
- board text added: "Make the holes for test points slightly bigger."
