File: h_bridge.kicad_sch (KiCad schematic)
At the start: 14 parts, among them J17 H-OUT, J18 Screw_Terminal_01x02, U10 TC118S

Commit message: Fixed CJC5340 C Number
Parts:
- J17: value H-OUT -> H OUT
- J18: value Screw_Terminal_01x02 -> - H IN +
Changed lines of the file:
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@@
 			)
 		)
-		(property "Value" "H-OUT"
+		(property "Value" "H OUT"
 			(at 182.88 81.2799 0)
 			(hide yes)
@@
 			)
 		)
-		(property "Value" "Screw_Terminal_01x02"
+		(property "Value" "- H IN +"
 			(at 182.88 36.8299 0)
-			(hide yes)
-			(show_name no)
-			(do_not_autoplace no)
+			(show_name no)
+			(do_not_autoplace no)
