File: si5351a.kicad_sch (KiCad schematic)
At the start: 11 parts, among them J8 BNC, U4 MS5351M

Commit message: Getting JLCPCB Price
Parts:
- J8: value BNC -> CLK2
Changed lines of the file:
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@@
 			)
 		)
-		(property "Value" "BNC"
+		(property "Value" "CLK2"
 			(at 181.2926 114.3 0)
 			(effects

Commit message: Initial v0.2
Fixed SCL-SDA swap, 3V3 on encoder, and 3D models for Kicad 10
Parts:
- FB1, FB4: value ~ -> (none)

Commit message: started routing
Parts:
- removed J8: CLK2, Connector_Coaxial:BNC_TEConnectivity_1478204_Vertical, symbol Connector:Conn_Coaxial
- added C34, C91: 10uF, PCM_JLCPCB:C_1206, symbol PCM_JLCPCB-Capacitors:1206,10uF
- added C84: 100uF, PCM_JLCPCB:C_CASE-B-3528-21(mm), symbol PCM_JLCPCB-Capacitors:CASE-B-3528-21(mm),100uF
- added JP7: Jumper_3_Bridged12, Jumper:SolderJumper-3_P1.3mm_Bridged12_RoundedPad1.0x1.5mm_NumberLabels, symbol Jumper:Jumper_3_Bridged12
- added JP8: Jumper_3_Bridged12, Jumper:SolderJumper-3_P1.3mm_Bridged12_RoundedPad1.0x1.5mm, symbol Jumper:Jumper_3_Bridged12
- added R72: 33Ω, PCM_JLCPCB:R_0805, symbol PCM_JLCPCB-Resistors:0805,33Ω
- added R74: 1Ω, PCM_JLCPCB:R_0805, symbol PCM_JLCPCB-Resistors:0805,1Ω
- added U11: SN74LVC74ADR, Package_SO:SOIC-14_3.9x8.7mm_P1.27mm, symbol 74xx:74LS74
Connections:
- net +3.3V: now also C84.1, R74.2; no longer FB1.1, FB4.2
- net CLK_0: now also TP3.1
- net CLK_1: now also TP4.1
- net GND: now also C34.2, C84.2, C91.2, U11.7 (GND)
- net 3.3VAO: now reaches C38.2, FB1.2, U4.7 (VDDO)
- net 3.3VAO: now also C91.1, U11.1 (~{R}), U11.10 (~{S}), U11.13 (~{R}), U11.14 (VCC), U11.4 (~{S})
- net at C15.2, FB4.1, U4.1 (VDD): now also C34.1
- net CLK2: no longer names the net of TP5.1, U4.6 (CLK2)
- net CLK2: now also R72.2
- new net: FB1.1, R74.1
- new net: R72.1, U11.11 (C), U11.3 (C)
- new net: U11.12 (D), U11.5 (Q)
- new net: U11.2 (D), U11.8 (~{Q})
- new net: JP8.1 (A), U11.9 (Q)
- new net: JP7.3 (B), U4.10 (CLK0)
- new net: JP8.3 (B), U4.9 (CLK1)
- new net: JP7.2 (C), R37.2
- new net: JP8.2 (C), R38.2
- new net: JP7.1 (A), U11.6 (~{Q})
- new net +3.3VA: FB4.2
Other:
- note added: "Johnson Counter for Quadrature"
- note added: "Lay this out so the Johnson counter is right next to the MS5351a, or move the 33 Ohm resistors close to each possible driver for the I and Q clocks."
- moved on the sheet: R37, R38

Commit message: Placed the second ADC
Parts:
- C15, C34, C38, C91: Manufacturer Samsung Electro-Mechanics -> (none)
- C84: Manufacturer AVX -> (none)
- FB1, FB4: Manufacturer Sunlord -> (none)
- R37, R38, R72, R74: Manufacturer UNI-ROYAL(Uniroyal Elec) -> (none)
- TP3, TP4, TP5: footprint TestPoint:TestPoint_THTPad_D1.5mm_Drill0.7mm -> TestPoint:TestPoint_THTPad_D2.0mm_Drill1.0mm
Changed lines of the file:
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@@
 			)
 		)
-		(property "Footprint" "TestPoint:TestPoint_THTPad_D1.5mm_Drill0.7mm"
+		(property "Footprint" "TestPoint:TestPoint_THTPad_D2.0mm_Drill1.0mm"
 			(at 255.27 102.87 0)
 			(hide yes)
@@
 			)
 		)
-		(property "Footprint" "TestPoint:TestPoint_THTPad_D1.5mm_Drill0.7mm"
+		(property "Footprint" "TestPoint:TestPoint_THTPad_D2.0mm_Drill1.0mm"
 			(at 161.29 118.11 0)
 			(hide yes)
@@
 			)
 		)
-		(property "Manufacturer" "Sunlord"
-			(at 142.24 87.63 0)
-			(hide yes)
-			(show_name no)
-			(do_not_autoplace no)
-			(effects
-				(font
-					(size 1.27 1.27)
-				)
-			)
-		)
 		(property "Part" "GZ2012D101TF"
 			(at 142.24 87.63 0)
@@
 			)
 		)
-		(property "Manufacturer" "AVX"
-			(at 152.4 73.66 0)
-			(hide yes)
-			(show_name no)
-			(do_not_autoplace no)
-			(effects
-				(font
-					(size 1.27 1.27)
-				)
-			)
-		)
 		(property "Part" "TAJB107K006RNJ"
 			(at 152.4 73.66 0)
@@
 			)
 		)
-		(property "Manufacturer" "Samsung Electro-Mechanics"
-			(at 151.13 95.25 0)
-			(hide yes)
-			(show_name no)
-			(do_not_autoplace no)
-			(effects
-				(font
-					(size 1.27 1.27)
-				)
-			)
-		)
 		(property "Part" "CL21B104KCFNNNE"
 			(at 151.13 95.25 0)
@@
 			)
 		)
-		(property "Manufacturer" "UNI-ROYAL(Uniroyal Elec)"
-			(at 245.11 102.87 0)
-			(hide yes)
-			(show_name no)
-			(do_not_autoplace no)
-			(effects
-				(font
-					(size 1.27 1.27)
-				)
-			)
-		)
 		(property "Part" "0805W8F330JT5E"
 			(at 245.11 102.87 0)
@@
 			)
 		)
-		(property "Manufacturer" "UNI-ROYAL(Uniroyal Elec)"
-			(at 245.11 118.11 0)
-			(hide yes)
-			(show_name no)
-			(do_not_autoplace no)
-			(effects
-				(font
-					(size 1.27 1.27)
-				)
-			)
-		)
 		(property "Part" "0805W8F330JT5E"
 			(at 245.11 118.11 0)
@@
 			)
 		)
-		(property "Footprint" "TestPoint:TestPoint_THTPad_D1.5mm_Drill0.7mm"
+		(property "Footprint" "TestPoint:TestPoint_THTPad_D2.0mm_Drill1.0mm"
 			(at 255.27 118.11 0)
 			(hide yes)
@@
 			)
 		)
-		(property "Manufacturer" "Samsung Electro-Mechanics"
-			(at 161.29 95.25 0)
-			(hide yes)
-			(show_name no)
-			(do_not_autoplace no)
-			(effects
-				(font
-					(size 1.27 1.27)
-				)
-			)
-		)
 		(property "Part" "CL31A106KBHNNNE"
 			(at 161.29 95.25 0)
@@
 			)
 		)
-		(property "Manufacturer" "Sunlord"
-			(at 137.16 83.82 0)
-			(hide yes)
-			(show_name no)
-			(do_not_autoplace no)
-			(effects
-				(font
-					(size 1.27 1.27)
-				)
-			)
-		)
 		(property "Part" "GZ2012D101TF"
 			(at 137.16 83.82 0)
@@
 			)
 		)
-		(property "Manufacturer" "UNI-ROYAL(Uniroyal Elec)"
-			(at 142.24 77.47 0)
-			(hide yes)
-			(show_name no)
-			(do_not_autoplace no)
-			(effects
-				(font
-					(size 1.27 1.27)
-				)
-			)
-		)
 		(property "Part" "0805W8F100KT5E"
 			(at 142.24 77.47 0)
@@
 			)
 		)
-		(property "Manufacturer" "UNI-ROYAL(Uniroyal Elec)"
-			(at 161.29 118.11 0)
-			(hide yes)
-			(show_name no)
-			(do_not_autoplace no)
-			(effects
-				(font
-					(size 1.27 1.27)
-				)
-			)
-		)
 		(property "Part" "0805W8F330JT5E"
 			(at 161.29 118.11 0)
@@
 			)
 		)
-		(property "Manufacturer" "Samsung Electro-Mechanics"
-			(at 128.27 93.98 0)
-			(hide yes)
-			(show_name no)
-			(do_not_autoplace no)
-			(effects
-				(font
-					(size 1.27 1.27)
-				)
-			)
-		)
 		(property "Part" "CL21B104KCFNNNE"
 			(at 128.27 93.98 0)
@@
 			(at 114.3 93.98 0)
 			(hide yes)
-			(show_name no)
-			(do_not_autoplace no)
-			(effects
-				(font
-					(size 1.27 1.27)
-				)
-			)
-		)
-		(property "Manufacturer" "Samsung Electro-Mechanics"
-			(at 114.3 93.98 0)
-			(hide yes)

Commit message: More routing
Parts:
- TP3, TP4, TP5: footprint TestPoint:TestPoint_THTPad_D2.0mm_Drill1.0mm -> TP_Label:TestPoint_THTPad_D2.0mm_Drill1.0mm
Changed lines of the file:
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@@
 			)
 		)
-		(property "Footprint" "TestPoint:TestPoint_THTPad_D2.0mm_Drill1.0mm"
+		(property "Footprint" "TP_Label:TestPoint_THTPad_D2.0mm_Drill1.0mm"
 			(at 255.27 102.87 0)
 			(hide yes)
@@
 			)
 		)
-		(property "Footprint" "TestPoint:TestPoint_THTPad_D2.0mm_Drill1.0mm"
+		(property "Footprint" "TP_Label:TestPoint_THTPad_D2.0mm_Drill1.0mm"
 			(at 161.29 118.11 0)
 			(hide yes)
@@
 			)
 		)
-		(property "Footprint" "TestPoint:TestPoint_THTPad_D2.0mm_Drill1.0mm"
+		(property "Footprint" "TP_Label:TestPoint_THTPad_D2.0mm_Drill1.0mm"
 			(at 255.27 118.11 0)
 			(hide yes)

Commit message: Fixed sub-schematic versions
Parts:
- JP7, JP8: value Jumper_3_Bridged12 -> Johnson?
Changed lines of the file:
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@@
 			)
 		)
-		(property "Value" "Jumper_3_Bridged12"
+		(property "Value" "Johnson?"
 			(at 226.06 116.8401 90)
 			(hide yes)
@@
 			)
 		)
-		(property "Value" "Jumper_3_Bridged12"
+		(property "Value" "Johnson?"
 			(at 226.06 104.1399 90)
 			(hide yes)

Commit message: Fixed CJC5340 C Number
Parts:
- JP7: value Johnson? -> Johnson Counter?
- JP8: value Johnson? -> Johnson Counter?; footprint Jumper:SolderJumper-3_P1.3mm_Bridged12_RoundedPad1.0x1.5mm -> Jumper:SolderJumper-3_P1.3mm_Bridged12_RoundedPad1.0x1.5mm_NumberLabels
Changed lines of the file:
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@@
 			)
 		)
-		(property "Value" "Johnson?"
-			(at 226.06 116.8401 90)
-			(hide yes)
+		(property "Value" "Johnson Counter?"
+			(at 247.396 114.554 90)
 			(show_name no)
 			(do_not_autoplace no)
@@
 			)
 		)
-		(property "Footprint" "Jumper:SolderJumper-3_P1.3mm_Bridged12_RoundedPad1.0x1.5mm"
+		(property "Footprint" "Jumper:SolderJumper-3_P1.3mm_Bridged12_RoundedPad1.0x1.5mm_NumberLabels"
 			(at 228.6 118.11 0)
 			(hide yes)
@@
 			)
 		)
-		(property "Value" "Johnson?"
+		(property "Value" "Johnson Counter?"
 			(at 226.06 104.1399 90)
 			(hide yes)
