File: pcm1808.kicad_sch (KiCad schematic)
At the start: 24 parts, among them J1 ADC IN, U2 PCM1808PWR

Commit message: Added CJC5340
Connections:
- net OUT_R: now reaches C7.1, R3.2, U2.14 (VINR)
- net OUT_L: now reaches C6.1, R2.2, U2.13 (VINL)
Changed lines of the file:
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@@
+		)
+	)
+	(hierarchical_label "OUT_R"
+		(shape output)
+		(at 130.81 91.44 0)
+		(effects
+			(font
+				(size 1.27 1.27)
+			)
+			(justify left)
 		)
 	)
@@
 		(effects
 			(font
+				(size 1.27 1.27)
+			)
+			(justify left)
+		)
+	)
+	(hierarchical_label "OUT_L"
+		(shape output)
+		(at 130.81 60.96 0)
+		(effects
+			(font

Commit message: Placed the second ADC
Parts:
- C10, C11, C13, C3, C4, C51, C6, C7: Manufacturer Samsung Electro-Mechanics -> (none)
- C44, C8, C9: Manufacturer AVX -> (none)
- R14, R16, R17, R18, R2, R3: Manufacturer UNI-ROYAL(Uniroyal Elec) -> (none)
- TP1, TP2: footprint TestPoint:TestPoint_THTPad_D1.5mm_Drill0.7mm -> TestPoint:TestPoint_THTPad_D2.0mm_Drill1.0mm
Changed lines of the file:
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@@
 			)
 		)
-		(property "Footprint" "TestPoint:TestPoint_THTPad_D1.5mm_Drill0.7mm"
+		(property "Footprint" "TestPoint:TestPoint_THTPad_D2.0mm_Drill1.0mm"
 			(at 86.36 67.31 0)
 			(hide yes)
@@
 			)
 		)
-		(property "Manufacturer" "Samsung Electro-Mechanics"
-			(at 167.64 55.88 0)
-			(hide yes)
-			(show_name no)
-			(do_not_autoplace no)
-			(effects
-				(font
-					(size 1.27 1.27)
-				)
-			)
-		)
 		(property "Part" "CL21B104KCFNNNE"
 			(at 167.64 55.88 0)
@@
 			)
 		)
-		(property "Manufacturer" "UNI-ROYAL(Uniroyal Elec)"
-			(at 115.57 91.44 0)
-			(hide yes)
-			(show_name no)
-			(do_not_autoplace no)
-			(effects
-				(font
-					(size 1.27 1.27)
-				)
-			)
-		)
 		(property "Part" "0603WAF4300T5E"
 			(at 115.57 91.44 0)
@@
 			)
 		)
-		(property "Manufacturer" "UNI-ROYAL(Uniroyal Elec)"
-			(at 227.33 92.71 0)
-			(hide yes)
-			(show_name no)
-			(do_not_autoplace no)
-			(effects
-				(font
-					(size 1.27 1.27)
-				)
-			)
-		)
 		(property "Part" "0805W8F330JT5E"
 			(at 227.33 92.71 0)
@@
 			)
 		)
-		(property "Manufacturer" "AVX"
-			(at 147.32 86.36 0)
-			(hide yes)
-			(show_name no)
-			(do_not_autoplace no)
-			(effects
-				(font
-					(size 1.27 1.27)
-				)
-			)
-		)
 		(property "Part" "TAJA106K016RNJ"
 			(at 147.32 86.36 0)
@@
 			)
 		)
-		(property "Manufacturer" "Samsung Electro-Mechanics"
-			(at 124.46 64.77 0)
-			(hide yes)
-			(show_name no)
-			(do_not_autoplace no)
-			(effects
-				(font
-					(size 1.27 1.27)
-				)
-			)
-		)
 		(property "Part" "CL21C222JBFNNNE"
 			(at 124.46 64.77 0)
@@
 			)
 		)
-		(property "Manufacturer" "AVX"
-			(at 161.29 55.88 0)
-			(hide yes)
-			(show_name no)
-			(do_not_autoplace no)
-			(effects
-				(font
-					(size 1.27 1.27)
-				)
-			)
-		)
 		(property "Part" "TAJA106K016RNJ"
 			(at 161.29 55.88 0)
@@
 			)
 		)
-		(property "Manufacturer" "Samsung Electro-Mechanics"
-			(at 59.69 85.09 0)
-			(hide yes)
-			(show_name no)
-			(do_not_autoplace no)
-			(effects
-				(font
-					(size 1.27 1.27)
-				)
-			)
-		)
 		(property "Part" "CL21B104KCFNNNE"
 			(at 59.69 85.09 0)
@@
 			)
 		)
-		(property "Manufacturer" "UNI-ROYAL(Uniroyal Elec)"
-			(at 227.33 95.25 0)
-			(hide yes)
-			(show_name no)
-			(do_not_autoplace no)
-			(effects
-				(font
-					(size 1.27 1.27)
-				)
-			)
-		)
 		(property "Part" "0805W8F330JT5E"
 			(at 227.33 95.25 0)
@@
 			)
 		)
-		(property "Manufacturer" "AVX"
-			(at 144.78 63.5 0)
-			(hide yes)
-			(show_name no)
-			(do_not_autoplace no)
-			(effects
-				(font
-					(size 1.27 1.27)
-				)
-			)
-		)
 		(property "Part" "TAJA106K016RNJ"
 			(at 144.78 63.5 0)
@@
 			)
 		)
-		(property "Manufacturer" "Samsung Electro-Mechanics"
-			(at 151.13 63.5 0)
-			(hide yes)
-			(show_name no)
-			(do_not_autoplace no)
-			(effects
-				(font
-					(size 1.27 1.27)
-				)
-			)
-		)
 		(property "Part" "CL21B104KCFNNNE"
 			(at 151.13 63.5 0)
@@
 			)
 		)
-		(property "Manufacturer" "Samsung Electro-Mechanics"
-			(at 96.52 67.31 0)
-			(hide yes)
-			(show_name no)
-			(do_not_autoplace no)
-			(effects
-				(font
-					(size 1.27 1.27)
-				)
-			)
-		)
 		(property "Part" "CL21B105KBFNNNE"
 			(at 96.52 67.31 0)
@@
 			)
 		)
-		(property "Manufacturer" "Samsung Electro-Mechanics"
-			(at 96.52 86.36 0)
-			(hide yes)
-			(show_name no)
-			(do_not_autoplace no)
-			(effects
-				(font
-					(size 1.27 1.27)
-				)
-			)
-		)
 		(property "Part" "CL21B105KBFNNNE"
 			(at 96.52 86.36 0)
@@
 			)
 		)
-		(property "Manufacturer" "Samsung Electro-Mechanics"
-			(at 124.46 95.25 0)
-			(hide yes)
-			(show_name no)
-			(do_not_autoplace no)
-			(effects
-				(font
-					(size 1.27 1.27)
-				)
-			)
-		)
 		(property "Part" "CL21C222JBFNNNE"
 			(at 124.46 95.25 0)
@@
 			)
 		)
-		(property "Footprint" "TestPoint:TestPoint_THTPad_D1.5mm_Drill0.7mm"
+		(property "Footprint" "TestPoint:TestPoint_THTPad_D2.0mm_Drill1.0mm"
 			(at 76.2 69.85 0)
 			(hide yes)
@@
 			)
 		)
-		(property "Manufacturer" "UNI-ROYAL(Uniroyal Elec)"
-			(at 115.57 60.96 0)
-			(hide yes)
-			(show_name no)
-			(do_not_autoplace no)
-			(effects
-				(font
-					(size 1.27 1.27)
-				)
-			)
-		)
 		(property "Part" "0603WAF4300T5E"
 			(at 115.57 60.96 0)
@@
 			)
 		)
-		(property "Manufacturer" "UNI-ROYAL(Uniroyal Elec)"
-			(at 227.33 97.79 0)
-			(hide yes)
-			(show_name no)
-			(do_not_autoplace no)
-			(effects
-				(font
-					(size 1.27 1.27)
-				)
-			)
-		)
 		(property "Part" "0805W8F330JT5E"
 			(at 227.33 97.79 0)
@@
 			)
 		)
-		(property "Manufacturer" "UNI-ROYAL(Uniroyal Elec)"
-			(at 63.5 85.09 0)
-			(hide yes)
-			(show_name no)
-			(do_not_autoplace no)
-			(effects
-				(font
-					(size 1.27 1.27)
-				)
-			)
-		)
 		(property "Part" "0603WAF100JT5E"
 			(at 63.5 85.09 0)
@@
 			(at 153.67 86.36 0)
 			(hide yes)
-			(show_name no)
-			(do_not_autoplace no)
-			(effects
-				(font
-					(size 1.27 1.27)
-				)
-			)
-		)
-		(property "Manufacturer" "Samsung Electro-Mechanics"
-			(at 153.67 86.36 0)
-			(hide yes)

Commit message: More routing
Parts:
- TP1, TP2: footprint TestPoint:TestPoint_THTPad_D2.0mm_Drill1.0mm -> TP_Label:TestPoint_THTPad_D2.0mm_Drill1.0mm
Changed lines of the file:
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@@
 			)
 		)
-		(property "Footprint" "TestPoint:TestPoint_THTPad_D2.0mm_Drill1.0mm"
+		(property "Footprint" "TP_Label:TestPoint_THTPad_D2.0mm_Drill1.0mm"
 			(at 86.36 67.31 0)
 			(hide yes)
@@
 			)
 		)
-		(property "Footprint" "TestPoint:TestPoint_THTPad_D2.0mm_Drill1.0mm"
+		(property "Footprint" "TP_Label:TestPoint_THTPad_D2.0mm_Drill1.0mm"
 			(at 76.2 69.85 0)
 			(hide yes)

Commit message: Fixing jumper labels and missing wire
Parts:
- JP19: value GND_LP_SND -> Q->ADC
Changed lines of the file:
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@@
 			)
 		)
-		(property "Value" "GND_LP_SND"
+		(property "Value" "Q->ADC"
 			(at 111.76 100.33 90)
 			(hide yes)

Commit message: I->ADC  Label
Parts:
- JP18: value GND_LP_SND -> I->ADC
Changed lines of the file:
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@@
 			)
 		)
-		(property "Value" "GND_LP_SND"
+		(property "Value" "I->ADC"
 			(at 111.76 55.88 90)
 			(hide yes)

Commit message: Input circuit for the CJT5340
Parts:
- removed C3, C4: 1uF, PCM_JLCPCB:C_0805, symbol PCM_JLCPCB-Capacitors:0805,1uF
- added C54, C56: 10uF, PCM_JLCPCB:C_CASE-A-3216-18(mm), symbol PCM_JLCPCB-Capacitors:CASE-A-3216-18(mm),10uF
Connections:
- net at J1.R, TP1.1: now also C54.1
- net at J1.T, TP2.1: now also C56.1
- net at JP19.2 (B), R3.1: now also C56.2
- net at JP18.1 (A), R2.1: now also C54.2

Commit message: R43 and R44 to 100 Ohms
Parts:
- removed R2, R3: 430Ω, PCM_JLCPCB:R_0603, symbol PCM_JLCPCB-Resistors:0603,430Ω
- added R43, R44: 100Ω, PCM_JLCPCB:R_0603, symbol PCM_JLCPCB-Resistors:0603,100Ω
Connections:
- net OUT_L: now also R43.2
- net OUT_R: now also R44.2
- net at C56.2, JP19.2 (B): now also R44.1
- net at C54.2, JP18.1 (A): now also R43.1
