File: CJC5340.kicad_sch (KiCad schematic)
At the start: 22 parts

Commit message: fixed version and page type
Other:
- note added: "Leave this out next time!"
Changed lines of the file:
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@@
+		)
+	)
+	(text "Leave this out next time!"
+		(exclude_from_sim no)
+		(at 121.158 143.256 0)
+		(effects
+			(font
+				(size 1.27 1.27)
+			)
 		)
 	)
