File: Module_Joshua/Module_Joshua.kicad_sch (KiCad schematic)
At the start: 1 part, among them J1 HC-SR04 connector

Commit message: Imported Student Parts
Not using Project Instances yet.
Parts:
- renumbered J1 to J?
Changed lines of the file:
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@@
 		(dnp no)
 		(fields_autoplaced yes)
-		(property "Reference" "#PWR098"
+		(property "Reference" "#PWR?"
 			(at 184.15 107.95 0)
 			(effects
@@
 			(project ""
 				(path "/c12dc015-e6cb-468c-8de4-269c3106de0e/360bd6cb-8515-415a-b1e1-cedd8caa152c"
-					(reference "#PWR098")
+					(reference "#PWR?")
 					(unit 1)
 				)
@@
 		(dnp no)
 		(fields_autoplaced yes)
-		(property "Reference" "#PWR099"
+		(property "Reference" "#PWR?"
 			(at 184.15 97.79 0)
 			(effects
@@
 			(project "Intro-to-CAD-2026"
 				(path "/c12dc015-e6cb-468c-8de4-269c3106de0e/360bd6cb-8515-415a-b1e1-cedd8caa152c"
-					(reference "#PWR099")
+					(reference "#PWR?")
 					(unit 1)
 				)
@@
 		(on_board yes)
 		(dnp no)
-		(property "Reference" "J1"
+		(property "Reference" "J?"
 			(at 168.91 107.95 0)
 			(effects
@@
 			(project ""
 				(path "/c12dc015-e6cb-468c-8de4-269c3106de0e/360bd6cb-8515-415a-b1e1-cedd8caa152c"
-					(reference "J1")
+					(reference "J?")
 					(unit 1)
 				)

Commit message: Going to school.
Parts:
- gave numbers to parts that had none: 1
Changed lines of the file:
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@@
 		(dnp no)
 		(fields_autoplaced yes)
-		(property "Reference" "#PWR?"
+		(property "Reference" "#PWR0116"
 			(at 184.15 107.95 0)
 			(effects
@@
 			(project ""
 				(path "/c12dc015-e6cb-468c-8de4-269c3106de0e/360bd6cb-8515-415a-b1e1-cedd8caa152c"
-					(reference "#PWR?")
+					(reference "#PWR0116")
 					(unit 1)
 				)
@@
 		(dnp no)
 		(fields_autoplaced yes)
-		(property "Reference" "#PWR?"
+		(property "Reference" "#PWR0115"
 			(at 184.15 97.79 0)
 			(effects
@@
 			(project "Intro-to-CAD-2026"
 				(path "/c12dc015-e6cb-468c-8de4-269c3106de0e/360bd6cb-8515-415a-b1e1-cedd8caa152c"
-					(reference "#PWR?")
+					(reference "#PWR0115")
 					(unit 1)
 				)
@@
 		(on_board yes)
 		(dnp no)
-		(property "Reference" "J?"
+		(property "Reference" "J6"
 			(at 168.91 107.95 0)
 			(effects
@@
 					(size 1.27 1.27)
 				)
-				(hide yes)
 			)
 		)
@@
 			(project ""
 				(path "/c12dc015-e6cb-468c-8de4-269c3106de0e/360bd6cb-8515-415a-b1e1-cedd8caa152c"
-					(reference "J?")
+					(reference "J6")
 					(unit 1)
 				)

Commit message: No Errors No Warnings
Some were excluded.
Parts:
- J6: footprint Connector_PinHeader_2.54mm:PinHeader_1x04_P2.54mm_Vertical -> Connector_PinSocket_2.54mm:PinSocket_1x04_P2.54mm_Vertical
Changed lines of the file:
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@@
 	)
 	(hierarchical_label "ECHO"
-		(shape input)
+		(shape output)
 		(at 184.15 99.06 0)
 		(effects
@@
 	)
 	(symbol
+		(lib_id "Connector_Generic:Conn_01x04")
+		(at 168.91 96.52 0)
+		(mirror y)
+		(unit 1)
+		(exclude_from_sim no)
+		(in_bom yes)
+		(on_board yes)
+		(dnp no)
+		(property "Reference" "J6"
+			(at 168.91 107.95 0)
+			(effects
+				(font
+					(size 1.27 1.27)
+				)
+			)
+		)
+		(property "Value" "HC-SR04 connector"
+			(at 169.164 90.678 0)
+			(effects
+				(font
+					(size 1.27 1.27)
+				)
+			)
+		)
+		(property "Footprint" "Connector_PinSocket_2.54mm:PinSocket_1x04_P2.54mm_Vertical"
+			(at 168.91 96.52 0)
+			(effects
+				(font
+					(size 1.27 1.27)
+				)
+				(hide yes)
+			)
+		)
+		(property "Datasheet" "https://www.makerguides.com/hc-sr04-arduino-tutorial/"
+			(at 168.91 96.52 0)
+			(effects
+				(font
+					(size 1.27 1.27)
+				)
+				(hide yes)
+			)
+		)
+		(property "Description" "Generic connector, single row, 01x04, script generated (kicad-library-utils/schlib/autogen/connector/)"
+			(at 168.91 96.52 0)
+			(effects
+				(font
+					(size 1.27 1.27)
+				)
+				(hide yes)
+			)
+		)
+		(pin "4"
+		)
+		(pin "1"
+		)
+		(pin "2"
+		)
+		(pin "3"
+		)
+		(instances
+			(project "Intro-to-CAD-2026"
+				(path "/c12dc015-e6cb-468c-8de4-269c3106de0e/360bd6cb-8515-415a-b1e1-cedd8caa152c"
+					(reference "J6")
+					(unit 1)
+				)
+			)
+		)
+	)
+	(symbol
 		(lib_id "power:+3.3V")
 		(at 184.15 93.98 0)
@@
 					(unit 1)
 				)
-			)
-		)
-	)
-	(symbol
-		(lib_id "Connector_Generic:Conn_01x04")
-		(at 168.91 96.52 0)
-		(mirror y)
-		(unit 1)
-		(exclude_from_sim no)
-		(in_bom yes)
-		(on_board yes)
-		(dnp no)
-		(property "Reference" "J6"
-			(at 168.91 107.95 0)
-			(effects
-				(font
-					(size 1.27 1.27)
-				)
-			)
-		)
-		(property "Value" "HC-SR04 connector"
-			(at 169.164 90.678 0)
-			(effects
-				(font
-					(size 1.27 1.27)
-				)
-			)
-		)
-		(property "Footprint" "Connector_PinHeader_2.54mm:PinHeader_1x04_P2.54mm_Vertical"
-			(at 168.91 96.52 0)
-			(effects
-				(font
-					(size 1.27 1.27)
-				)
-				(hide yes)
-			)
-		)
-		(property "Datasheet" "~"
-			(at 168.91 96.52 0)
-			(effects
-				(font
-					(size 1.27 1.27)
-				)
-				(hide yes)
-			)
-		)
-		(property "Description" "Generic connector, single row, 01x04, script generated (kicad-library-utils/schlib/autogen/connector/)"
-			(at 168.91 96.52 0)
-			(effects
-				(font
-					(size 1.27 1.27)
-				)
-				(hide yes)
-			)
-		)
-		(pin "4"
-		)
-		(pin "1"
-		)
-		(pin "2"
-		)
-		(pin "3"
-		)
-		(instances
-			(project ""
-				(path "/c12dc015-e6cb-468c-8de4-269c3106de0e/360bd6cb-8515-415a-b1e1-cedd8caa152c"
-					(reference "J6")
-					(unit 1)
-				)
-			)
-			(project ""
-				(path "/ea0c559e-3bae-46d5-a508-0445335e2a4b"
-					(reference "J1")
-					(unit 1)
-				)

Commit message: Getting JLCPCB Price
Parts:
- J6: value HC-SR04 connector -> HC-SR04; LCSC (none) -> C2718488
Changed lines of the file:
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@@
 			)
 		)
-		(property "Value" "HC-SR04 connector"
+		(property "Value" "HC-SR04"
 			(at 169.164 90.678 0)
 			(effects
@@
 			(at 168.91 96.52 0)
 			(effects
+				(font
+					(size 1.27 1.27)
+				)
+				(hide yes)
+			)
+		)
+		(property "LCSC" "C2718488"
+			(at 168.91 96.52 0)
+			(effects
