File: Module_KyleS/Module_KyleS.kicad_sch (KiCad schematic)
At the start: 8 parts, among them J1 Micro_SD-TF_PUSH

Commit message: Imported Student Parts
Not using Project Instances yet.
Parts:
- renumbered C1 to C?, C2 to C?, J1 to J?, R5 to R?, R2 to R?, R3 to R?, R1 to R?, R4 to R?
Changed lines of the file:
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@@
 		(dnp no)
 		(fields_autoplaced yes)
-		(property "Reference" "R5"
+		(property "Reference" "R?"
 			(at 184.15 111.7599 0)
 			(effects
@@
 			(project "Module_Template"
 				(path "/c12dc015-e6cb-468c-8de4-269c3106de0e/1d172d86-7589-4f73-960e-a08dc80ef343"
-					(reference "R5")
+					(reference "R?")
 					(unit 1)
 				)
@@
 		(dnp no)
 		(fields_autoplaced yes)
-		(property "Reference" "#PWR083"
+		(property "Reference" "#PWR?"
 			(at 123.19 71.12 0)
 			(effects
@@
 			(project "Module_Template"
 				(path "/c12dc015-e6cb-468c-8de4-269c3106de0e/1d172d86-7589-4f73-960e-a08dc80ef343"
-					(reference "#PWR083")
+					(reference "#PWR?")
 					(unit 1)
 				)
@@
 		(on_board yes)
 		(dnp no)
-		(property "Reference" "C1"
+		(property "Reference" "C?"
 			(at 115.57 69.8499 0)
 			(effects
@@
 			(project "Module_Template"
 				(path "/c12dc015-e6cb-468c-8de4-269c3106de0e/1d172d86-7589-4f73-960e-a08dc80ef343"
-					(reference "C1")
+					(reference "C?")
 					(unit 1)
 				)
@@
 		(on_board yes)
 		(dnp no)
-		(property "Reference" "R2"
+		(property "Reference" "R?"
 			(at 89.662 96.52 0)
 			(effects
@@
 			(project "Module_Template"
 				(path "/c12dc015-e6cb-468c-8de4-269c3106de0e/1d172d86-7589-4f73-960e-a08dc80ef343"
-					(reference "R2")
+					(reference "R?")
 					(unit 1)
 				)
@@
 		(dnp no)
 		(fields_autoplaced yes)
-		(property "Reference" "#PWR087"
+		(property "Reference" "#PWR?"
 			(at 181.61 109.22 0)
 			(effects
@@
 			(project "Module_Template"
 				(path "/c12dc015-e6cb-468c-8de4-269c3106de0e/1d172d86-7589-4f73-960e-a08dc80ef343"
-					(reference "#PWR087")
+					(reference "#PWR?")
 					(unit 1)
 				)
@@
 		(on_board yes)
 		(dnp no)
-		(property "Reference" "R3"
+		(property "Reference" "R?"
 			(at 100.838 96.52 0)
 			(effects
@@
 			(project "Module_Template"
 				(path "/c12dc015-e6cb-468c-8de4-269c3106de0e/1d172d86-7589-4f73-960e-a08dc80ef343"
-					(reference "R3")
+					(reference "R?")
 					(unit 1)
 				)
@@
 		(on_board yes)
 		(dnp no)
-		(property "Reference" "J1"
+		(property "Reference" "J?"
 			(at 159.385 82.55 0)
 			(effects
@@
 			(project "Module_Template"
 				(path "/c12dc015-e6cb-468c-8de4-269c3106de0e/1d172d86-7589-4f73-960e-a08dc80ef343"
-					(reference "J1")
+					(reference "J?")
 					(unit 1)
 				)
@@
 		(dnp no)
 		(fields_autoplaced yes)
-		(property "Reference" "#PWR084"
+		(property "Reference" "#PWR?"
 			(at 146.05 134.62 0)
 			(effects
@@
 			(project "Module_Template"
 				(path "/c12dc015-e6cb-468c-8de4-269c3106de0e/1d172d86-7589-4f73-960e-a08dc80ef343"
-					(reference "#PWR084")
+					(reference "#PWR?")
 					(unit 1)
 				)
@@
 		(on_board yes)
 		(dnp no)
-		(property "Reference" "R1"
+		(property "Reference" "R?"
 			(at 80.518 96.52 0)
 			(effects
@@
 			(project "Module_Template"
 				(path "/c12dc015-e6cb-468c-8de4-269c3106de0e/1d172d86-7589-4f73-960e-a08dc80ef343"
-					(reference "R1")
+					(reference "R?")
 					(unit 1)
 				)
@@
 		(dnp no)
 		(fields_autoplaced yes)
-		(property "Reference" "#PWR085"
+		(property "Reference" "#PWR?"
 			(at 123.19 83.82 0)
 			(effects
@@
 			(project "Module_Template"
 				(path "/c12dc015-e6cb-468c-8de4-269c3106de0e/1d172d86-7589-4f73-960e-a08dc80ef343"
-					(reference "#PWR085")
+					(reference "#PWR?")
 					(unit 1)
 				)
@@
 		(dnp no)
 		(fields_autoplaced yes)
-		(property "Reference" "C2"
+		(property "Reference" "C?"
 			(at 130.81 69.8499 0)
 			(effects
@@
 			(project "Module_Template"
 				(path "/c12dc015-e6cb-468c-8de4-269c3106de0e/1d172d86-7589-4f73-960e-a08dc80ef343"
-					(reference "C2")
+					(reference "C?")
 					(unit 1)
 				)
@@
 		(dnp no)
 		(fields_autoplaced yes)
-		(property "Reference" "#PWR086"
+		(property "Reference" "#PWR?"
 			(at 95.25 91.44 0)
 			(effects
@@
 			(project "Module_Template"
 				(path "/c12dc015-e6cb-468c-8de4-269c3106de0e/1d172d86-7589-4f73-960e-a08dc80ef343"
-					(reference "#PWR086")
+					(reference "#PWR?")
 					(unit 1)
 				)
@@
 		(on_board yes)
 		(dnp no)
-		(property "Reference" "R4"
+		(property "Reference" "R?"
 			(at 109.982 96.52 0)
 			(effects
@@
 			(project "Module_Template"
 				(path "/c12dc015-e6cb-468c-8de4-269c3106de0e/1d172d86-7589-4f73-960e-a08dc80ef343"
-					(reference "R4")
-					(unit 1)
-				)
+					(reference "R?")
+					(unit 1)
+				)

Commit message: Going to school.
Parts:
- gave numbers to parts that had none: 8
Changed lines of the file:
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@@
 		(dnp no)
 		(fields_autoplaced yes)
-		(property "Reference" "R?"
+		(property "Reference" "R69"
 			(at 184.15 111.7599 0)
 			(effects
@@
 			(project "Module_Template"
 				(path "/c12dc015-e6cb-468c-8de4-269c3106de0e/1d172d86-7589-4f73-960e-a08dc80ef343"
-					(reference "R?")
+					(reference "R69")
 					(unit 1)
 				)
@@
 		(dnp no)
 		(fields_autoplaced yes)
-		(property "Reference" "#PWR?"
+		(property "Reference" "#PWR0118"
 			(at 123.19 71.12 0)
 			(effects
@@
 			(project "Module_Template"
 				(path "/c12dc015-e6cb-468c-8de4-269c3106de0e/1d172d86-7589-4f73-960e-a08dc80ef343"
-					(reference "#PWR?")
+					(reference "#PWR0118")
 					(unit 1)
 				)
@@
 		(on_board yes)
 		(dnp no)
-		(property "Reference" "C?"
+		(property "Reference" "C66"
 			(at 115.57 69.8499 0)
 			(effects
@@
 			(project "Module_Template"
 				(path "/c12dc015-e6cb-468c-8de4-269c3106de0e/1d172d86-7589-4f73-960e-a08dc80ef343"
-					(reference "C?")
+					(reference "C66")
 					(unit 1)
 				)
@@
 		(on_board yes)
 		(dnp no)
-		(property "Reference" "R?"
+		(property "Reference" "R66"
 			(at 89.662 96.52 0)
 			(effects
@@
 			(project "Module_Template"
 				(path "/c12dc015-e6cb-468c-8de4-269c3106de0e/1d172d86-7589-4f73-960e-a08dc80ef343"
-					(reference "R?")
+					(reference "R66")
 					(unit 1)
 				)
@@
 		(dnp no)
 		(fields_autoplaced yes)
-		(property "Reference" "#PWR?"
+		(property "Reference" "#PWR0124"
 			(at 181.61 109.22 0)
 			(effects
@@
 			(project "Module_Template"
 				(path "/c12dc015-e6cb-468c-8de4-269c3106de0e/1d172d86-7589-4f73-960e-a08dc80ef343"
-					(reference "#PWR?")
+					(reference "#PWR0124")
 					(unit 1)
 				)
@@
 		(on_board yes)
 		(dnp no)
-		(property "Reference" "R?"
+		(property "Reference" "R67"
 			(at 100.838 96.52 0)
 			(effects
@@
 			(project "Module_Template"
 				(path "/c12dc015-e6cb-468c-8de4-269c3106de0e/1d172d86-7589-4f73-960e-a08dc80ef343"
-					(reference "R?")
+					(reference "R67")
 					(unit 1)
 				)
@@
 		(on_board yes)
 		(dnp no)
-		(property "Reference" "J?"
+		(property "Reference" "J13"
 			(at 159.385 82.55 0)
 			(effects
@@
 			(project "Module_Template"
 				(path "/c12dc015-e6cb-468c-8de4-269c3106de0e/1d172d86-7589-4f73-960e-a08dc80ef343"
-					(reference "J?")
+					(reference "J13")
 					(unit 1)
 				)
@@
 		(dnp no)
 		(fields_autoplaced yes)
-		(property "Reference" "#PWR?"
+		(property "Reference" "#PWR0123"
 			(at 146.05 134.62 0)
 			(effects
@@
 			(project "Module_Template"
 				(path "/c12dc015-e6cb-468c-8de4-269c3106de0e/1d172d86-7589-4f73-960e-a08dc80ef343"
-					(reference "#PWR?")
+					(reference "#PWR0123")
 					(unit 1)
 				)
@@
 		(on_board yes)
 		(dnp no)
-		(property "Reference" "R?"
+		(property "Reference" "R65"
 			(at 80.518 96.52 0)
 			(effects
@@
 			(project "Module_Template"
 				(path "/c12dc015-e6cb-468c-8de4-269c3106de0e/1d172d86-7589-4f73-960e-a08dc80ef343"
-					(reference "R?")
+					(reference "R65")
 					(unit 1)
 				)
@@
 		(dnp no)
 		(fields_autoplaced yes)
-		(property "Reference" "#PWR?"
+		(property "Reference" "#PWR0119"
 			(at 123.19 83.82 0)
 			(effects
@@
 			(project "Module_Template"
 				(path "/c12dc015-e6cb-468c-8de4-269c3106de0e/1d172d86-7589-4f73-960e-a08dc80ef343"
-					(reference "#PWR?")
+					(reference "#PWR0119")
 					(unit 1)
 				)
@@
 		(dnp no)
 		(fields_autoplaced yes)
-		(property "Reference" "C?"
+		(property "Reference" "C67"
 			(at 130.81 69.8499 0)
 			(effects
@@
 			(project "Module_Template"
 				(path "/c12dc015-e6cb-468c-8de4-269c3106de0e/1d172d86-7589-4f73-960e-a08dc80ef343"
-					(reference "C?")
+					(reference "C67")
 					(unit 1)
 				)
@@
 		(dnp no)
 		(fields_autoplaced yes)
-		(property "Reference" "#PWR?"
+		(property "Reference" "#PWR0117"
 			(at 95.25 91.44 0)
 			(effects
@@
 			(project "Module_Template"
 				(path "/c12dc015-e6cb-468c-8de4-269c3106de0e/1d172d86-7589-4f73-960e-a08dc80ef343"
-					(reference "#PWR?")
+					(reference "#PWR0117")
 					(unit 1)
 				)
@@
 		(on_board yes)
 		(dnp no)
-		(property "Reference" "R?"
+		(property "Reference" "R68"
 			(at 109.982 96.52 0)
 			(effects
@@
 			(project "Module_Template"
 				(path "/c12dc015-e6cb-468c-8de4-269c3106de0e/1d172d86-7589-4f73-960e-a08dc80ef343"
-					(reference "R?")
-					(unit 1)
-				)
+					(reference "R68")
+					(unit 1)
+				)

Commit message: Placed the second ADC
Parts:
- C66: Manufacturer Samsung Electro-Mechanics -> (none)
- C67: Manufacturer YAGEO -> (none)
- R65, R66, R67, R68, R69: Manufacturer UNI-ROYAL(Uniroyal Elec) -> (none)
Changed lines of the file:
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@@
-			)
-		)
-		(property "Manufacturer" "UNI-ROYAL(Uniroyal Elec)"
-			(at 181.61 111.76 0)
-			(hide yes)
-			(show_name no)
-			(do_not_autoplace no)
-			(effects
-				(font
-					(size 1.27 1.27)
-				)
 			)
 		)
@@
 			)
 		)
-		(property "Manufacturer" "Samsung Electro-Mechanics"
-			(at 118.11 72.39 0)
-			(hide yes)
-			(show_name no)
-			(do_not_autoplace no)
-			(effects
-				(font
-					(size 1.27 1.27)
-				)
-			)
-		)
 		(property "Part" "CL21A106KAYNNNE"
 			(at 118.11 72.39 0)
@@
 			)
 		)
-		(property "Manufacturer" "UNI-ROYAL(Uniroyal Elec)"
-			(at 87.63 96.52 0)
-			(hide yes)
-			(show_name no)
-			(do_not_autoplace no)
-			(effects
-				(font
-					(size 1.27 1.27)
-				)
-			)
-		)
 		(property "Part" "0603WAF1002T5E"
 			(at 87.63 96.52 0)
@@
 			)
 		)
-		(property "Manufacturer" "UNI-ROYAL(Uniroyal Elec)"
-			(at 102.87 96.52 0)
-			(hide yes)
-			(show_name no)
-			(do_not_autoplace no)
-			(effects
-				(font
-					(size 1.27 1.27)
-				)
-			)
-		)
 		(property "Part" "0603WAF1002T5E"
 			(at 102.87 96.52 0)
@@
 			)
 		)
-		(property "Manufacturer" "UNI-ROYAL(Uniroyal Elec)"
-			(at 82.55 96.52 0)
-			(hide yes)
-			(show_name no)
-			(do_not_autoplace no)
-			(effects
-				(font
-					(size 1.27 1.27)
-				)
-			)
-		)
 		(property "Part" "0603WAF1002T5E"
 			(at 82.55 96.52 0)
@@
 			)
 		)
-		(property "Manufacturer" "YAGEO"
-			(at 128.27 72.39 0)
-			(hide yes)
-			(show_name no)
-			(do_not_autoplace no)
-			(effects
-				(font
-					(size 1.27 1.27)
-				)
-			)
-		)
 		(property "Part" "CC0603KRX7R9BB104"
 			(at 128.27 72.39 0)
@@
 			(at 107.95 96.52 0)
 			(hide yes)
-			(show_name no)
-			(do_not_autoplace no)
-			(effects
-				(font
-					(size 1.27 1.27)
-				)
-			)
-		)
-		(property "Manufacturer" "UNI-ROYAL(Uniroyal Elec)"
-			(at 107.95 96.52 0)
-			(hide yes)
