File: Module_Andre/Module_Andre.kicad_sch (KiCad schematic)
At the start: 7 parts, among them SW1 RotaryEncoder_Switch_MP

Commit message: Imported Student Parts
Not using Project Instances yet.
Parts:
- renumbered C3 to C?, C2 to C?, C1 to C?, R2 to R?, R3 to R?, R1 to R?, SW1 to SW?
Changed lines of the file:
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@@
 		(dnp no)
 		(fields_autoplaced yes)
-		(property "Reference" "#PWR07"
+		(property "Reference" "#PWR?"
 			(at 46.99 97.79 0)
 			(effects
@@
 			(project ""
 				(path "/c12dc015-e6cb-468c-8de4-269c3106de0e/1314eab6-d054-48f7-88b3-f0d5cb35f00b"
-					(reference "#PWR07")
+					(reference "#PWR?")
 					(unit 1)
 				)
@@
 		(dnp no)
 		(fields_autoplaced yes)
-		(property "Reference" "C3"
+		(property "Reference" "C?"
 			(at 69.85 83.8199 0)
 			(effects
@@
 			(project ""
 				(path "/c12dc015-e6cb-468c-8de4-269c3106de0e/1314eab6-d054-48f7-88b3-f0d5cb35f00b"
-					(reference "C3")
+					(reference "C?")
 					(unit 1)
 				)
@@
 		(dnp no)
 		(fields_autoplaced yes)
-		(property "Reference" "#PWR06"
+		(property "Reference" "#PWR?"
 			(at 31.75 29.21 0)
 			(effects
@@
 			(project ""
 				(path "/c12dc015-e6cb-468c-8de4-269c3106de0e/1314eab6-d054-48f7-88b3-f0d5cb35f00b"
-					(reference "#PWR06")
+					(reference "#PWR?")
 					(unit 1)
 				)
@@
 		(on_board yes)
 		(dnp no)
-		(property "Reference" "R2"
+		(property "Reference" "R?"
 			(at 49.53 71.1199 0)
 			(effects
@@
 			(project ""
 				(path "/c12dc015-e6cb-468c-8de4-269c3106de0e/1314eab6-d054-48f7-88b3-f0d5cb35f00b"
-					(reference "R2")
+					(reference "R?")
 					(unit 1)
 				)
@@
 		(dnp no)
 		(fields_autoplaced yes)
-		(property "Reference" "C2"
+		(property "Reference" "C?"
 			(at 49.53 83.8199 0)
 			(effects
@@
 			(project ""
 				(path "/c12dc015-e6cb-468c-8de4-269c3106de0e/1314eab6-d054-48f7-88b3-f0d5cb35f00b"
-					(reference "C2")
+					(reference "C?")
 					(unit 1)
 				)
@@
 		(dnp no)
 		(fields_autoplaced yes)
-		(property "Reference" "#PWR04"
+		(property "Reference" "#PWR?"
 			(at 46.99 69.85 0)
 			(effects
@@
 			(project ""
 				(path "/c12dc015-e6cb-468c-8de4-269c3106de0e/1314eab6-d054-48f7-88b3-f0d5cb35f00b"
-					(reference "#PWR04")
+					(reference "#PWR?")
 					(unit 1)
 				)
@@
 		(dnp no)
 		(fields_autoplaced yes)
-		(property "Reference" "C1"
+		(property "Reference" "C?"
 			(at 34.29 43.1799 0)
 			(effects
@@
 			(project ""
 				(path "/c12dc015-e6cb-468c-8de4-269c3106de0e/1314eab6-d054-48f7-88b3-f0d5cb35f00b"
-					(reference "C1")
+					(reference "C?")
 					(unit 1)
 				)
@@
 		(dnp no)
 		(fields_autoplaced yes)
-		(property "Reference" "#PWR08"
+		(property "Reference" "#PWR?"
 			(at 67.31 97.79 0)
 			(effects
@@
 			(project ""
 				(path "/c12dc015-e6cb-468c-8de4-269c3106de0e/1314eab6-d054-48f7-88b3-f0d5cb35f00b"
-					(reference "#PWR08")
+					(reference "#PWR?")
 					(unit 1)
 				)
@@
 		(dnp no)
 		(fields_autoplaced yes)
-		(property "Reference" "#PWR05"
+		(property "Reference" "#PWR?"
 			(at 67.31 69.85 0)
 			(effects
@@
 			(project ""
 				(path "/c12dc015-e6cb-468c-8de4-269c3106de0e/1314eab6-d054-48f7-88b3-f0d5cb35f00b"
-					(reference "#PWR05")
+					(reference "#PWR?")
 					(unit 1)
 				)
@@
 		(dnp no)
 		(fields_autoplaced yes)
-		(property "Reference" "SW1"
+		(property "Reference" "SW?"
 			(at 50.8 49.5299 90)
 			(effects
@@
 			(project "Module_Template"
 				(path "/c12dc015-e6cb-468c-8de4-269c3106de0e/1314eab6-d054-48f7-88b3-f0d5cb35f00b"
-					(reference "SW1")
+					(reference "SW?")
 					(unit 1)
 				)
@@
 		(dnp no)
 		(fields_autoplaced yes)
-		(property "Reference" "#PWR01"
+		(property "Reference" "#PWR?"
 			(at 57.15 97.79 0)
 			(effects
@@
 			(project ""
 				(path "/c12dc015-e6cb-468c-8de4-269c3106de0e/1314eab6-d054-48f7-88b3-f0d5cb35f00b"
-					(reference "#PWR01")
+					(reference "#PWR?")
 					(unit 1)
 				)
@@
 		(dnp no)
 		(fields_autoplaced yes)
-		(property "Reference" "R3"
+		(property "Reference" "R?"
 			(at 69.85 71.1199 0)
 			(effects
@@
 			(project ""
 				(path "/c12dc015-e6cb-468c-8de4-269c3106de0e/1314eab6-d054-48f7-88b3-f0d5cb35f00b"
-					(reference "R3")
+					(reference "R?")
 					(unit 1)
 				)
@@
 		(dnp no)
 		(fields_autoplaced yes)
-		(property "Reference" "#PWR03"
+		(property "Reference" "#PWR?"
 			(at 31.75 57.15 0)
 			(effects
@@
 			(project ""
 				(path "/c12dc015-e6cb-468c-8de4-269c3106de0e/1314eab6-d054-48f7-88b3-f0d5cb35f00b"
-					(reference "#PWR03")
+					(reference "#PWR?")
 					(unit 1)
 				)
@@
 		(dnp no)
 		(fields_autoplaced yes)
-		(property "Reference" "#PWR02"
+		(property "Reference" "#PWR?"
 			(at 82.55 60.96 0)
 			(effects
@@
 			(project ""
 				(path "/c12dc015-e6cb-468c-8de4-269c3106de0e/1314eab6-d054-48f7-88b3-f0d5cb35f00b"
-					(reference "#PWR02")
+					(reference "#PWR?")
 					(unit 1)
 				)
@@
 		(dnp no)
 		(fields_autoplaced yes)
-		(property "Reference" "R1"
+		(property "Reference" "R?"
 			(at 34.29 30.4799 0)
 			(effects
@@
 			(project ""
 				(path "/c12dc015-e6cb-468c-8de4-269c3106de0e/1314eab6-d054-48f7-88b3-f0d5cb35f00b"
-					(reference "R1")
-					(unit 1)
-				)
+					(reference "R?")
+					(unit 1)
+				)

Commit message: Going to school.
Parts:
- gave numbers to parts that had none: 7
Changed lines of the file:
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@@
 		(dnp no)
 		(fields_autoplaced yes)
-		(property "Reference" "#PWR?"
+		(property "Reference" "#PWR0110"
 			(at 46.99 97.79 0)
 			(effects
@@
 			(project ""
 				(path "/c12dc015-e6cb-468c-8de4-269c3106de0e/1314eab6-d054-48f7-88b3-f0d5cb35f00b"
-					(reference "#PWR?")
+					(reference "#PWR0110")
 					(unit 1)
 				)
@@
 		(dnp no)
 		(fields_autoplaced yes)
-		(property "Reference" "C?"
+		(property "Reference" "C65"
 			(at 69.85 83.8199 0)
 			(effects
@@
 			(project ""
 				(path "/c12dc015-e6cb-468c-8de4-269c3106de0e/1314eab6-d054-48f7-88b3-f0d5cb35f00b"
-					(reference "C?")
+					(reference "C65")
 					(unit 1)
 				)
@@
 		(dnp no)
 		(fields_autoplaced yes)
-		(property "Reference" "#PWR?"
+		(property "Reference" "#PWR098"
 			(at 31.75 29.21 0)
 			(effects
@@
 			(project ""
 				(path "/c12dc015-e6cb-468c-8de4-269c3106de0e/1314eab6-d054-48f7-88b3-f0d5cb35f00b"
-					(reference "#PWR?")
+					(reference "#PWR098")
 					(unit 1)
 				)
@@
 		(on_board yes)
 		(dnp no)
-		(property "Reference" "R?"
+		(property "Reference" "R63"
 			(at 49.53 71.1199 0)
 			(effects
@@
 			(project ""
 				(path "/c12dc015-e6cb-468c-8de4-269c3106de0e/1314eab6-d054-48f7-88b3-f0d5cb35f00b"
-					(reference "R?")
+					(reference "R63")
 					(unit 1)
 				)
@@
 		(dnp no)
 		(fields_autoplaced yes)
-		(property "Reference" "C?"
+		(property "Reference" "C64"
 			(at 49.53 83.8199 0)
 			(effects
@@
 			(project ""
 				(path "/c12dc015-e6cb-468c-8de4-269c3106de0e/1314eab6-d054-48f7-88b3-f0d5cb35f00b"
-					(reference "C?")
+					(reference "C64")
 					(unit 1)
 				)
@@
 		(dnp no)
 		(fields_autoplaced yes)
-		(property "Reference" "#PWR?"
+		(property "Reference" "#PWR0100"
 			(at 46.99 69.85 0)
 			(effects
@@
 			(project ""
 				(path "/c12dc015-e6cb-468c-8de4-269c3106de0e/1314eab6-d054-48f7-88b3-f0d5cb35f00b"
-					(reference "#PWR?")
+					(reference "#PWR0100")
 					(unit 1)
 				)
@@
 		(dnp no)
 		(fields_autoplaced yes)
-		(property "Reference" "C?"
+		(property "Reference" "C62"
 			(at 34.29 43.1799 0)
 			(effects
@@
 			(project ""
 				(path "/c12dc015-e6cb-468c-8de4-269c3106de0e/1314eab6-d054-48f7-88b3-f0d5cb35f00b"
-					(reference "C?")
+					(reference "C62")
 					(unit 1)
 				)
@@
 		(dnp no)
 		(fields_autoplaced yes)
-		(property "Reference" "#PWR?"
+		(property "Reference" "#PWR0113"
 			(at 67.31 97.79 0)
 			(effects
@@
 			(project ""
 				(path "/c12dc015-e6cb-468c-8de4-269c3106de0e/1314eab6-d054-48f7-88b3-f0d5cb35f00b"
-					(reference "#PWR?")
+					(reference "#PWR0113")
 					(unit 1)
 				)
@@
 		(dnp no)
 		(fields_autoplaced yes)
-		(property "Reference" "#PWR?"
+		(property "Reference" "#PWR0112"
 			(at 67.31 69.85 0)
 			(effects
@@
 			(project ""
 				(path "/c12dc015-e6cb-468c-8de4-269c3106de0e/1314eab6-d054-48f7-88b3-f0d5cb35f00b"
-					(reference "#PWR?")
+					(reference "#PWR0112")
 					(unit 1)
 				)
@@
 		(dnp no)
 		(fields_autoplaced yes)
-		(property "Reference" "SW?"
+		(property "Reference" "SW1"
 			(at 50.8 49.5299 90)
 			(effects
@@
 			(project "Module_Template"
 				(path "/c12dc015-e6cb-468c-8de4-269c3106de0e/1314eab6-d054-48f7-88b3-f0d5cb35f00b"
-					(reference "SW?")
+					(reference "SW1")
 					(unit 1)
 				)
@@
 		(dnp no)
 		(fields_autoplaced yes)
-		(property "Reference" "#PWR?"
+		(property "Reference" "#PWR0111"
 			(at 57.15 97.79 0)
 			(effects
@@
 			(project ""
 				(path "/c12dc015-e6cb-468c-8de4-269c3106de0e/1314eab6-d054-48f7-88b3-f0d5cb35f00b"
-					(reference "#PWR?")
+					(reference "#PWR0111")
 					(unit 1)
 				)
@@
 		(dnp no)
 		(fields_autoplaced yes)
-		(property "Reference" "R?"
+		(property "Reference" "R64"
 			(at 69.85 71.1199 0)
 			(effects
@@
 			(project ""
 				(path "/c12dc015-e6cb-468c-8de4-269c3106de0e/1314eab6-d054-48f7-88b3-f0d5cb35f00b"
-					(reference "R?")
+					(reference "R64")
 					(unit 1)
 				)
@@
 		(dnp no)
 		(fields_autoplaced yes)
-		(property "Reference" "#PWR?"
+		(property "Reference" "#PWR099"
 			(at 31.75 57.15 0)
 			(effects
@@
 			(project ""
 				(path "/c12dc015-e6cb-468c-8de4-269c3106de0e/1314eab6-d054-48f7-88b3-f0d5cb35f00b"
-					(reference "#PWR?")
+					(reference "#PWR099")
 					(unit 1)
 				)
@@
 		(dnp no)
 		(fields_autoplaced yes)
-		(property "Reference" "#PWR?"
+		(property "Reference" "#PWR0114"
 			(at 82.55 60.96 0)
 			(effects
@@
 			(project ""
 				(path "/c12dc015-e6cb-468c-8de4-269c3106de0e/1314eab6-d054-48f7-88b3-f0d5cb35f00b"
-					(reference "#PWR?")
+					(reference "#PWR0114")
 					(unit 1)
 				)
@@
 		(dnp no)
 		(fields_autoplaced yes)
-		(property "Reference" "R?"
+		(property "Reference" "R57"
 			(at 34.29 30.4799 0)
 			(effects
@@
 			(project ""
 				(path "/c12dc015-e6cb-468c-8de4-269c3106de0e/1314eab6-d054-48f7-88b3-f0d5cb35f00b"
-					(reference "R?")
-					(unit 1)
-				)
+					(reference "R57")
+					(unit 1)
+				)

Commit message: No Errors No Warnings
Some were excluded.
Changed lines of the file:
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@@
 	)
 	(hierarchical_label "GPIO_B"
-		(shape input)
+		(shape output)
 		(at 69.85 77.47 0)
 		(effects
@@
 	)
 	(hierarchical_label "GPIO_C"
-		(shape input)
+		(shape output)
 		(at 29.21 36.83 180)
 		(effects
@@
 	)
 	(hierarchical_label "GPIO_A"
-		(shape input)
+		(shape output)
 		(at 44.45 77.47 180)
 		(effects

Commit message: Initial v0.2
Fixed SCL-SDA swap, 3V3 on encoder, and 3D models for Kicad 10
Connections:
- net +3V3 renamed +3.3V

Commit message: Updated errors
Other:
- note added: "The +3.3V had the wrong label. This means they need to be jumped to +3.3V."
Changed lines of the file:
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@@
 	(generator_version "10.0")
 	(paper "A4")
+	(text "The +3.3V had the wrong label.  This means they need to be jumped to +3.3V."
+		(exclude_from_sim no)
+		(at 54.356 16.764 0)
+		(effects
+			(font
+				(size 1.27 1.27)
+				(color 255 0 52 1)
+			)
+		)
+	)
 	(junction
 		(at 31.75 39.37)

Commit message: Starting a new branch for v0.2
Other:
- note removed: "The +3.3V had the wrong label. This means they need to be jumped to +3.3V."
Changed lines of the file:
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@@
 	(generator_version "10.0")
 	(paper "A4")
-	(text "The +3.3V had the wrong label.  This means they need to be jumped to +3.3V."
-		(exclude_from_sim no)
-		(at 54.356 16.764 0)
-		(effects
-			(font
-				(size 1.27 1.27)
-				(color 255 0 52 1)
-			)
-		)
-	)
 	(junction
 		(at 31.75 39.37)

Commit message: Placed the second ADC
Parts:
- C62, C64, C65: Manufacturer Samsung Electro-Mechanics -> (none)
- R57, R63, R64: Manufacturer UNI-ROYAL(Uniroyal Elec) -> (none)
Changed lines of the file:
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@@
-			)
-		)
-		(property "Manufacturer" "Samsung Electro-Mechanics"
-			(at 67.31 86.36 0)
-			(hide yes)
-			(show_name no)
-			(do_not_autoplace no)
-			(effects
-				(font
-					(size 1.27 1.27)
-				)
 			)
 		)
@@
 		)
 		(property "Category" "Resistors,Chip Resistor - Surface Mount"
-			(at 46.99 71.12 0)
-			(hide yes)
-			(show_name no)
-			(do_not_autoplace no)
-			(effects
-				(font
-					(size 1.27 1.27)
-				)
-			)
-		)
-		(property "Manufacturer" "UNI-ROYAL(Uniroyal Elec)"
 			(at 46.99 71.12 0)
 			(hide yes)
@@
 			)
 		)
-		(property "Manufacturer" "Samsung Electro-Mechanics"
-			(at 46.99 86.36 0)
-			(hide yes)
-			(show_name no)
-			(do_not_autoplace no)
-			(effects
-				(font
-					(size 1.27 1.27)
-				)
-			)
-		)
 		(property "Part" "CL05B103KB5NNNC"
 			(at 46.99 86.36 0)
@@
 			)
 		)
-		(property "Manufacturer" "Samsung Electro-Mechanics"
-			(at 31.75 45.72 0)
-			(hide yes)
-			(show_name no)
-			(do_not_autoplace no)
-			(effects
-				(font
-					(size 1.27 1.27)
-				)
-			)
-		)
 		(property "Part" "CL05B104KB54PNC"
 			(at 31.75 45.72 0)
@@
 		)
 		(property "Category" "Resistors,Chip Resistor - Surface Mount"
-			(at 67.31 71.12 0)
-			(hide yes)
-			(show_name no)
-			(do_not_autoplace no)
-			(effects
-				(font
-					(size 1.27 1.27)
-				)
-			)
-		)
-		(property "Manufacturer" "UNI-ROYAL(Uniroyal Elec)"
 			(at 67.31 71.12 0)
 			(hide yes)
@@
 			(at 31.75 30.48 0)
 			(hide yes)
-			(show_name no)
-			(do_not_autoplace no)
-			(effects
-				(font
-					(size 1.27 1.27)
-				)
-			)
-		)
-		(property "Manufacturer" "UNI-ROYAL(Uniroyal Elec)"
-			(at 31.75 30.48 0)
-			(hide yes)
