File: v0.2/Hardware/Intro-to-CAD-2026.kicad_sch (KiCad schematic)
At the start: 9 parts

Commit message: Fix Module References in v0.2
Other:
- sheet Angle_Encoder: file Module_Andre/Module_Andre.kicad_sch -> Module_Andre.kicad_sch
- sheet LED String: file Module_JaronGarbi/Module_JaronGarbi.kicad_sch -> Module_JaronGarbi.kicad_sch
- sheet Push Button: file Module_Micah/Module_Micah.kicad_sch -> Module_Micah.kicad_sch
- sheet SPI_MicroSD: file Module_KyleS/Module_KyleS.kicad_sch -> Module_KyleS.kicad_sch
- sheet Ultrasound_Distance: file Module_Joshua/Module_Joshua.kicad_sch -> Module_Joshua.kicad_sch
Changed lines of the file:
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@@
 			)
 		)
-		(property "Sheetfile" "Module_Andre/Module_Andre.kicad_sch"
+		(property "Sheetfile" "Module_Andre.kicad_sch"
 			(at 124.46 50.1146 0)
 			(show_name no)
@@
 			)
 		)
-		(property "Sheetfile" "Module_KyleS/Module_KyleS.kicad_sch"
+		(property "Sheetfile" "Module_KyleS.kicad_sch"
 			(at 124.46 100.9146 0)
 			(show_name no)
@@
 			)
 		)
-		(property "Sheetfile" "Module_Joshua/Module_Joshua.kicad_sch"
+		(property "Sheetfile" "Module_Joshua.kicad_sch"
 			(at 124.46 72.9746 0)
 			(show_name no)
@@
 			)
 		)
-		(property "Sheetfile" "Module_JaronGarbi/Module_JaronGarbi.kicad_sch"
+		(property "Sheetfile" "Module_JaronGarbi.kicad_sch"
 			(at 125.73 149.1746 0)
 			(show_name no)
@@
 			)
 		)
-		(property "Sheetfile" "Module_Micah/Module_Micah.kicad_sch"
+		(property "Sheetfile" "Module_Micah.kicad_sch"
 			(at 124.46 127.5846 0)
 			(show_name no)
