File: v0.2/Hardware/qsd-sdr.kicad_sch (KiCad schematic)
At the start: 57 parts, among them J11 SDR ANT, J12 SDR Out, U5 OPA1612AxD, U7 SN74CBT3253DBQR, U8 OPA1612AxD

Commit message: Added Soapy README
Other:
- note added: "We should switch X this transformer so the choke is on the input, though this way is giving us a 6 dB gain we would lose with the choke on the input."
- note removed: "We should switch X this transformer so the choke is on the input."
Changed lines of the file:
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@@
 		(rev "0.2")
 	)
-	(text "We should switch X this transformer\nso the choke is on the input."
+	(text "We should switch X this transformer\nso the choke is on the input, though\nthis way is giving us a 6 dB gain we\nwould lose with the choke on the input."
 		(exclude_from_sim no)
 		(at 89.154 57.912 0)
