File: v0.1/Hardware/Module_Andre.kicad_sch (KiCad schematic)
At the start: 11 parts, among them J8 CLK2, U4 MS5351M

Commit message: Fixed modules in v0.1
Parts:
- removed C15, C38: 100nF, PCM_JLCPCB:C_0805, symbol PCM_JLCPCB-Capacitors:0805,100nF
- removed FB1, FB4: (no value), PCM_JLCPCB:FB_0805, symbol PCM_JLCPCB-Inductors:Ferrite,0805
- removed J8: CLK2, Connector_Coaxial:BNC_TEConnectivity_1478204_Vertical, symbol Connector:Conn_Coaxial
- removed R37, R38: 33Ω, PCM_JLCPCB:R_0805, symbol PCM_JLCPCB-Resistors:0805,33Ω
- removed TP3: I LO, TestPoint:TestPoint_THTPad_D1.5mm_Drill0.7mm, symbol Connector:TestPoint
- removed TP4: Q LO, TestPoint:TestPoint_THTPad_D1.5mm_Drill0.7mm, symbol Connector:TestPoint
- removed TP5: OSC, TestPoint:TestPoint_THTPad_D1.5mm_Drill0.7mm, symbol Connector:TestPoint
- removed U4: MS5351M, Package_SO:MSOP-10_3x3mm_P0.5mm, symbol Oscillator:Si5351A-B-GT
- added C62: 100nF, PCM_JLCPCB:C_0402, symbol PCM_JLCPCB-Capacitors:0402,100nF,(2)
- added C64, C65: 10nF, PCM_JLCPCB:C_0402, symbol PCM_JLCPCB-Capacitors:0402,10nF
- added R57, R63, R64: 10kΩ, PCM_JLCPCB:R_0402, symbol PCM_JLCPCB-Resistors:0402,10kΩ
- added SW1: RotaryEncoder_Switch_MP, Rotary_Encoder:RotaryEncoder_Alps_EC11E-Switch_Vertical_H20mm, symbol Device:RotaryEncoder_Switch_MP
Connections:
- net +3.3V: now also R57.1, R63.1, R64.1
- net GND: now also C62.2, C64.2, C65.2, SW1.C, SW1.MP, SW1.S2
- new net GPIO_A: C64.1, R63.2, SW1.A
- new net GPIO_B: C65.1, R64.2, SW1.B
- new net GPIO_C: C62.1, R57.2, SW1.S1
- no-connect marks 1 -> 0
Other:
- note removed: "24.576 MHz"
- note removed: "Oscillator"
